File: Main PCB KiCAD/squid.kicad_sch (KiCad schematic)
At the start: 3 parts, among them U3 ESP32-S2-WROVER

Commit message: battery charging
Parts:
- R4: value 1k -> 330
Connections:
- net +5V is gone; now on net +3.3V: R4.1
- net +3.3V: now reaches U3.2 (3V3)
Changed lines of the file:
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@@
 	)
 	(symbol
-		(lib_id "power:+5V")
-		(at 204.47 101.6 0)
-		(unit 1)
-		(exclude_from_sim no)
-		(in_bom yes)
-		(on_board yes)
-		(dnp no)
-		(fields_autoplaced yes)
-		(property "Reference" "#PWR020"
-			(at 204.47 105.41 0)
-			(effects
-				(font
-					(size 1.27 1.27)
-				)
-				(hide yes)
-			)
-		)
-		(property "Value" "+5V"
-			(at 204.47 96.52 0)
+		(lib_id "power:+3.3V")
+		(at 80.01 59.69 0)
+		(unit 1)
+		(exclude_from_sim no)
+		(in_bom yes)
+		(on_board yes)
+		(dnp no)
+		(property "Reference" "#PWR011"
+			(at 80.01 63.5 0)
+			(effects
+				(font
+					(size 1.27 1.27)
+				)
+				(hide yes)
+			)
+		)
+		(property "Value" "+3.3V"
+			(at 80.391 55.2958 0)
 			(effects
 				(font
@@
 		)
 		(property "Footprint" ""
-			(at 204.47 101.6 0)
+			(at 80.01 59.69 0)
 			(effects
 				(font
@@
 		)
 		(property "Datasheet" ""
-			(at 204.47 101.6 0)
-			(effects
-				(font
-					(size 1.27 1.27)
-				)
-				(hide yes)
-			)
-		)
-		(property "Description" "Power symbol creates a global label with name \"+5V\""
-			(at 204.47 101.6 0)
-			(effects
-				(font
-					(size 1.27 1.27)
-				)
-				(hide yes)
+			(at 80.01 59.69 0)
+			(effects
+				(font
+					(size 1.27 1.27)
+				)
+				(hide yes)
+			)
+		)
+		(property "Description" ""
+			(at 80.01 59.69 0)
+			(effects
+				(font
+					(size 1.27 1.27)
+				)
 			)
 		)
@@
 			(project "Buoy PCB"
 				(path "/a041e2a6-7d41-458c-91f3-753821d3dfe9/b1b5818c-3c6a-4a38-a6f8-0a964c6bc0f0"
-					(reference "#PWR020")
+					(reference "#PWR011")
 					(unit 1)
 				)
@@
 	)
 	(symbol
+		(lib_id "power:+3.3V")
+		(at 204.47 101.6 0)
+		(unit 1)
+		(exclude_from_sim no)
+		(in_bom yes)
+		(on_board yes)
+		(dnp no)
+		(property "Reference" "#PWR012"
+			(at 204.47 105.41 0)
+			(effects
+				(font
+					(size 1.27 1.27)
+				)
+				(hide yes)
+			)
+		)
+		(property "Value" "+3.3V"
+			(at 204.851 97.2058 0)
+			(effects
+				(font
+					(size 1.27 1.27)
+				)
+			)
+		)
+		(property "Footprint" ""
+			(at 204.47 101.6 0)
+			(effects
+				(font
+					(size 1.27 1.27)
+				)
+				(hide yes)
+			)
+		)
+		(property "Datasheet" ""
+			(at 204.47 101.6 0)
+			(effects
+				(font
+					(size 1.27 1.27)
+				)
+				(hide yes)
+			)
+		)
+		(property "Description" ""
+			(at 204.47 101.6 0)
+			(effects
+				(font
+					(size 1.27 1.27)
+				)
+			)
+		)
+		(pin "1"
+		)
+		(instances
+			(project "Buoy PCB"
+				(path "/a041e2a6-7d41-458c-91f3-753821d3dfe9/b1b5818c-3c6a-4a38-a6f8-0a964c6bc0f0"
+					(reference "#PWR012")
+					(unit 1)
+				)
+			)
+		)
+	)
+	(symbol
 		(lib_id "RF_Module:ESP32-S2-WROVER")
 		(at 80.01 90.17 0)
@@
 			)
 		)
-		(property "Value" "1k"
+		(property "Value" "330"
 			(at 207.01 107.9499 0)
 			(effects

Commit message: this is likely to break all the things…
Connections:
- net +3.3V: now also D2.2 (A); no longer R4.1
- net GND: now also R4.2; no longer D2.1 (K)
- new net: D2.1 (K), R4.1
Other:
- moved on the sheet: D2, R4
Changed lines of the file:
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@@
 	(symbol
 		(lib_id "Device:R_Small")
-		(at 204.47 106.68 0)
+		(at 204.47 114.3 0)
 		(unit 1)
 		(exclude_from_sim no)
@@
 		(fields_autoplaced yes)
 		(property "Reference" "R4"
-			(at 207.01 105.4099 0)
+			(at 207.01 113.0299 0)
 			(effects
 				(font
@@
 		)
 		(property "Value" "330"
-			(at 207.01 107.9499 0)
+			(at 207.01 115.5699 0)
 			(effects
 				(font
@@
 		)
 		(property "Footprint" "Resistor_SMD:R_0805_2012Metric_Pad1.20x1.40mm_HandSolder"
-			(at 204.47 106.68 0)
+			(at 204.47 114.3 0)
 			(effects
 				(font
@@
 		)
 		(property "Datasheet" "~"
-			(at 204.47 106.68 0)
+			(at 204.47 114.3 0)
 			(effects
 				(font
@@
 		)
 		(property "Description" "Resistor, small symbol"
-			(at 204.47 106.68 0)
+			(at 204.47 114.3 0)
 			(effects
 				(font
@@
 	(symbol
 		(lib_id "Device:LED_Small_Filled")
-		(at 204.47 114.3 90)
+		(at 204.47 106.68 90)
 		(unit 1)
 		(exclude_from_sim no)
@@
 		(fields_autoplaced yes)
 		(property "Reference" "D2"
-			(at 207.01 112.9664 90)
+			(at 207.01 105.3464 90)
 			(effects
 				(font
@@
 		)
 		(property "Value" "RED"
-			(at 207.01 115.5064 90)
+			(at 207.01 107.8864 90)
 			(effects
 				(font
@@
 		)
 		(property "Footprint" "LED_SMD:LED_0805_2012Metric_Pad1.15x1.40mm_HandSolder"
-			(at 204.47 114.3 90)
+			(at 204.47 106.68 90)
 			(effects
 				(font
@@
 		)
 		(property "Datasheet" "~"
-			(at 204.47 114.3 90)
+			(at 204.47 106.68 90)
 			(effects
 				(font
@@
 		)
 		(property "Description" "Light emitting diode, small symbol, filled shape"
-			(at 204.47 114.3 0)
+			(at 204.47 106.68 0)
 			(effects
 				(font
@@
 		)
 		(property "Sim.Pins" "1=K 2=A"
-			(at 204.47 114.3 0)
+			(at 204.47 106.68 0)
 			(effects
 				(font

Commit message: clean
Connections:
- net +3.3V: now also R4.1; no longer D2.2 (A)
- net GND: now also D2.1 (K); no longer R4.2
- new net: D2.2 (A), R4.2
Other:
- moved on the sheet: D2, R4
Changed lines of the file:
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@@
 	(symbol
 		(lib_id "Device:R_Small")
-		(at 204.47 114.3 0)
+		(at 204.47 106.68 0)
 		(unit 1)
 		(exclude_from_sim no)
@@
 		(fields_autoplaced yes)
 		(property "Reference" "R4"
-			(at 207.01 113.0299 0)
+			(at 207.01 105.4099 0)
 			(effects
 				(font
@@
 		)
 		(property "Value" "330"
-			(at 207.01 115.5699 0)
+			(at 207.01 107.9499 0)
 			(effects
 				(font
@@
 		)
 		(property "Footprint" "Resistor_SMD:R_0805_2012Metric_Pad1.20x1.40mm_HandSolder"
-			(at 204.47 114.3 0)
+			(at 204.47 106.68 0)
 			(effects
 				(font
@@
 		)
 		(property "Datasheet" "~"
-			(at 204.47 114.3 0)
+			(at 204.47 106.68 0)
 			(effects
 				(font
@@
 		)
 		(property "Description" "Resistor, small symbol"
-			(at 204.47 114.3 0)
+			(at 204.47 106.68 0)
 			(effects
 				(font
@@
 	(symbol
 		(lib_id "Device:LED_Small_Filled")
-		(at 204.47 106.68 90)
+		(at 204.47 114.3 90)
 		(unit 1)
 		(exclude_from_sim no)
@@
 		(fields_autoplaced yes)
 		(property "Reference" "D2"
-			(at 207.01 105.3464 90)
+			(at 207.01 112.9664 90)
 			(effects
 				(font
@@
 		)
 		(property "Value" "RED"
-			(at 207.01 107.8864 90)
+			(at 207.01 115.5064 90)
 			(effects
 				(font
@@
 		)
 		(property "Footprint" "LED_SMD:LED_0805_2012Metric_Pad1.15x1.40mm_HandSolder"
-			(at 204.47 106.68 90)
+			(at 204.47 114.3 90)
 			(effects
 				(font
@@
 		)
 		(property "Datasheet" "~"
-			(at 204.47 106.68 90)
+			(at 204.47 114.3 90)
 			(effects
 				(font
@@
 		)
 		(property "Description" "Light emitting diode, small symbol, filled shape"
-			(at 204.47 106.68 0)
+			(at 204.47 114.3 0)
 			(effects
 				(font
@@
 		)
 		(property "Sim.Pins" "1=K 2=A"
-			(at 204.47 106.68 0)
+			(at 204.47 114.3 0)
 			(effects
 				(font
