File: Main PCB KiCAD/solar.kicad_sch (KiCad schematic)
At the start: 18 parts, among them J2 Solar 1, J3 Solar 2, J4 Solar 3, J5 Solar 4, J6 Solar 5, J7 Solar 6, J8 Solar PCB

Commit message: battery charging
Parts:
- removed D3, D4, D5, D6, D7, D8: RB550VM-30TE-17, Diode_SMD:D_SOD-323_HandSoldering, symbol Device:D_Small_Filled
- removed J8: Solar PCB, Connector_Molex:Molex_Nano-Fit_105309-xx08_1x08_P2.50mm_Vertical, symbol Connector_Generic:Conn_01x08
- removed JP3: Solar - GND, Jumper:SolderJumper-2_P1.3mm_Bridged_RoundedPad1.0x1.5mm, symbol Jumper:SolderJumper_2_Bridged
- added D10, D3, D4, D5, D6, D7: 1N5819HW-FDICT, Diode_SMD:D_SOD-123, symbol Device:D_Schottky_Small_Filled
- R8, R9: value 1k -> 10k
Connections:
- net -Solar is gone; now on net GND: D9.1 (K), J2.2 (Pin_2), J3.2 (Pin_2), J4.2 (Pin_2), J5.2 (Pin_2), J6.2 (Pin_2), J7.2 (Pin_2), R9.2
- net +Solar: now also D10.1 (K), D3.1 (K), D4.1 (K), D5.1 (K), D6.1 (K), D7.1 (K)
- net at J7.1 (Pin_1): now also D5.2 (A)
- net at J2.1 (Pin_1): now also D10.2 (A)
- net at J4.1 (Pin_1): now also D4.2 (A)
- net at J3.1 (Pin_1): now also D3.2 (A)
- net at J6.1 (Pin_1): now also D6.2 (A)
- net at J5.1 (Pin_1): now also D7.2 (A)

Commit message: this is likely to break all the things…
Parts:
- removed J2: Solar 1, Connector_Molex:Molex_Nano-Fit_105309-xx02_1x02_P2.50mm_Vertical, symbol Connector_Generic:Conn_01x02
- removed J3: Solar 2, Connector_Molex:Molex_Nano-Fit_105309-xx02_1x02_P2.50mm_Vertical, symbol Connector_Generic:Conn_01x02
- removed J4: Solar 3, Connector_Molex:Molex_Nano-Fit_105309-xx02_1x02_P2.50mm_Vertical, symbol Connector_Generic:Conn_01x02
- removed J5: Solar 4, Connector_Molex:Molex_Nano-Fit_105309-xx02_1x02_P2.50mm_Vertical, symbol Connector_Generic:Conn_01x02
- removed J6: Solar 5, Connector_Molex:Molex_Nano-Fit_105309-xx02_1x02_P2.50mm_Vertical, symbol Connector_Generic:Conn_01x02
- removed J7: Solar 6, Connector_Molex:Molex_Nano-Fit_105309-xx02_1x02_P2.50mm_Vertical, symbol Connector_Generic:Conn_01x02
- added J8: Solar, Connector_Molex:Molex_Nano-Fit_105309-xx08_1x08_P2.50mm_Vertical, symbol Connector_Generic:Conn_01x08
Connections:
- net +Solar: now also D9.2 (A); no longer R7.1
- net GND: now also R7.2, J8.7 (Pin_7), J8.8 (Pin_8); no longer D9.1 (K)
- net at D4.2 (A): now also J8.5 (Pin_5)
- net at D7.2 (A): now also J8.2 (Pin_2)
- net at D5.2 (A): now also J8.4 (Pin_4)
- net at D3.2 (A): now also J8.6 (Pin_6)
- net at D6.2 (A): now also J8.3 (Pin_3)
- net at D10.2 (A): now also J8.1 (Pin_1)
- new net: D9.1 (K), R7.1
Other:
- moved on the sheet: D10, D3, D4, D5, D6, D7, D9, R7

Commit message: clean
Parts:
- removed D10: 1N5819HW-FDICT, Diode_SMD:D_SOD-123, symbol Device:D_Schottky_Small_Filled
- removed J8: Solar, Connector_Molex:Molex_Nano-Fit_105309-xx08_1x08_P2.50mm_Vertical, symbol Connector_Generic:Conn_01x08
- added D1: 1N5819HW-FDICT, Diode_SMD:D_SOD-123, symbol Device:D_Schottky_Small_Filled
- added J11: Conn_01x12_Socket, Connector_PinSocket_2.54mm:PinSocket_1x12_P2.54mm_Vertical, symbol Connector:Conn_01x12_Socket
Connections:
- net at D7.2 (A): now also J11.11 (Pin_11)
- net at D6.2 (A): now also J11.9 (Pin_9)
- net at D5.2 (A): now also J11.7 (Pin_7)
- net at D4.2 (A): now also J11.5 (Pin_5)
- net at D3.2 (A): now also J11.3 (Pin_3)
- net +Solar_Batt: now reaches R7.1
- net +Solar_Batt: now also D3.1 (K), D4.1 (K), D5.1 (K), D6.1 (K), D7.1 (K), R8.1, D1.1 (K); no longer D9.1 (K)
- removed net +Solar: D3.1 (K), D4.1 (K), D5.1 (K), D6.1 (K), D7.1 (K), D9.2 (A), R8.1
- net GND: no longer names the net of R7.2
- net GND: now also D9.2 (A); no longer R9.2
- new net: D1.2 (A), J11.1 (Pin_1)
- new net GND_Batt: D9.1 (K), J11.10 (Pin_10), J11.12 (Pin_12), J11.2 (Pin_2), J11.4 (Pin_4), J11.6 (Pin_6), J11.8 (Pin_8), R9.2
Other:
- moved on the sheet: D3, D4, D5, D6, D7, D9, R7

Commit message: update
Parts:
- renumbered D9 to D3, D1 to D4, D3 to D5, D4 to D6, D5 to D7, D6 to D8, D7 to D9, J11 to J9, R7 to R10
Changed lines of the file:
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@@
 		(dnp no)
 		(fields_autoplaced yes)
-		(property "Reference" "#PWR016"
+		(property "Reference" "#PWR035"
 			(at 99.06 64.77 0)
 			(effects
@@
 			(project "Buoy PCB"
 				(path "/a041e2a6-7d41-458c-91f3-753821d3dfe9/e8f4d549-a7ac-4e6a-bad9-8d4daf54a22c"
-					(reference "#PWR016")
+					(reference "#PWR035")
 					(unit 1)
 				)
@@
 		(on_board yes)
 		(dnp no)
-		(property "Reference" "D4"
+		(property "Reference" "D6"
 			(at 233.68 60.5536 0)
 			(effects
@@
 			(project "Buoy PCB"
 				(path "/a041e2a6-7d41-458c-91f3-753821d3dfe9/e8f4d549-a7ac-4e6a-bad9-8d4daf54a22c"
-					(reference "D4")
+					(reference "D6")
 					(unit 1)
 				)
@@
 		(on_board yes)
 		(dnp no)
-		(property "Reference" "D7"
+		(property "Reference" "D9"
 			(at 233.68 75.7936 0)
 			(effects
@@
 			(project "Buoy PCB"
 				(path "/a041e2a6-7d41-458c-91f3-753821d3dfe9/e8f4d549-a7ac-4e6a-bad9-8d4daf54a22c"
-					(reference "D7")
+					(reference "D9")
 					(unit 1)
 				)
@@
 		(on_board yes)
 		(dnp no)
-		(property "Reference" "D5"
+		(property "Reference" "D7"
 			(at 233.68 65.6336 0)
 			(effects
@@
 			(project "Buoy PCB"
 				(path "/a041e2a6-7d41-458c-91f3-753821d3dfe9/e8f4d549-a7ac-4e6a-bad9-8d4daf54a22c"
-					(reference "D5")
+					(reference "D7")
 					(unit 1)
 				)
@@
 		(on_board yes)
 		(dnp no)
-		(property "Reference" "J11"
+		(property "Reference" "J9"
 			(at 221.615 86.36 0)
 			(effects
@@
 			(project "Buoy PCB"
 				(path "/a041e2a6-7d41-458c-91f3-753821d3dfe9/e8f4d549-a7ac-4e6a-bad9-8d4daf54a22c"
-					(reference "J11")
+					(reference "J9")
 					(unit 1)
 				)
@@
 		(dnp no)
 		(fields_autoplaced yes)
-		(property "Reference" "#PWR036"
+		(property "Reference" "#PWR040"
 			(at 243.84 57.15 0)
 			(effects
@@
 			(project "Buoy PCB"
 				(path "/a041e2a6-7d41-458c-91f3-753821d3dfe9/e8f4d549-a7ac-4e6a-bad9-8d4daf54a22c"
-					(reference "#PWR036")
+					(reference "#PWR040")
 					(unit 1)
 				)
@@
 		(on_board yes)
 		(dnp no)
-		(property "Reference" "D3"
+		(property "Reference" "D5"
 			(at 233.68 55.4736 0)
 			(effects
@@
 			(project "Buoy PCB"
 				(path "/a041e2a6-7d41-458c-91f3-753821d3dfe9/e8f4d549-a7ac-4e6a-bad9-8d4daf54a22c"
-					(reference "D3")
+					(reference "D5")
 					(unit 1)
 				)
@@
 		(dnp no)
 		(fields_autoplaced yes)
-		(property "Reference" "#PWR031"
+		(property "Reference" "#PWR037"
 			(at 116.84 64.77 0)
 			(effects
@@
 			(project "Buoy PCB"
 				(path "/a041e2a6-7d41-458c-91f3-753821d3dfe9/e8f4d549-a7ac-4e6a-bad9-8d4daf54a22c"
-					(reference "#PWR031")
+					(reference "#PWR037")
 					(unit 1)
 				)
@@
 		(dnp no)
 		(fields_autoplaced yes)
-		(property "Reference" "#PWR013"
+		(property "Reference" "#PWR038"
 			(at 116.84 87.63 0)
 			(effects
@@
 			(project "Buoy PCB"
 				(path "/a041e2a6-7d41-458c-91f3-753821d3dfe9/e8f4d549-a7ac-4e6a-bad9-8d4daf54a22c"
-					(reference "#PWR013")
+					(reference "#PWR038")
 					(unit 1)
 				)
@@
 		(dnp no)
 		(fields_autoplaced yes)
-		(property "Reference" "#PWR017"
+		(property "Reference" "#PWR036"
 			(at 99.06 87.63 0)
 			(effects
@@
 			(project "Buoy PCB"
 				(path "/a041e2a6-7d41-458c-91f3-753821d3dfe9/e8f4d549-a7ac-4e6a-bad9-8d4daf54a22c"
-					(reference "#PWR017")
+					(reference "#PWR036")
 					(unit 1)
 				)
@@
 		(dnp no)
 		(fields_autoplaced yes)
-		(property "Reference" "R7"
+		(property "Reference" "R10"
 			(at 119.38 64.7699 0)
 			(effects
@@
 			(project "Buoy PCB"
 				(path "/a041e2a6-7d41-458c-91f3-753821d3dfe9/e8f4d549-a7ac-4e6a-bad9-8d4daf54a22c"
-					(reference "R7")
+					(reference "R10")
 					(unit 1)
 				)
@@
 		(dnp no)
 		(fields_autoplaced yes)
-		(property "Reference" "D9"
+		(property "Reference" "D3"
 			(at 119.38 74.8664 90)
 			(effects
@@
 			(project "Buoy PCB"
 				(path "/a041e2a6-7d41-458c-91f3-753821d3dfe9/e8f4d549-a7ac-4e6a-bad9-8d4daf54a22c"
-					(reference "D9")
+					(reference "D3")
 					(unit 1)
 				)
@@
 		(on_board yes)
 		(dnp no)
-		(property "Reference" "D1"
+		(property "Reference" "D4"
 			(at 233.68 50.3936 0)
 			(effects
@@
 			(project "Buoy PCB"
 				(path "/a041e2a6-7d41-458c-91f3-753821d3dfe9/e8f4d549-a7ac-4e6a-bad9-8d4daf54a22c"
-					(reference "D1")
+					(reference "D4")
 					(unit 1)
 				)
@@
 		(on_board yes)
 		(dnp no)
-		(property "Reference" "D6"
+		(property "Reference" "D8"
 			(at 233.68 70.7136 0)
 			(effects
@@
 			(project "Buoy PCB"
 				(path "/a041e2a6-7d41-458c-91f3-753821d3dfe9/e8f4d549-a7ac-4e6a-bad9-8d4daf54a22c"
-					(reference "D6")
+					(reference "D8")
 					(unit 1)
 				)
@@
 		(dnp no)
 		(fields_autoplaced yes)
-		(property "Reference" "#PWR014"
+		(property "Reference" "#PWR039"
 			(at 228.6 92.71 0)
 			(effects
@@
 			(project "Buoy PCB"
 				(path "/a041e2a6-7d41-458c-91f3-753821d3dfe9/e8f4d549-a7ac-4e6a-bad9-8d4daf54a22c"
-					(reference "#PWR014")
-					(unit 1)
-				)
+					(reference "#PWR039")
+					(unit 1)
+				)

Commit message: cleanup
Parts:
- added C2: 1u, Capacitor_SMD:C_0805_2012Metric_Pad1.18x1.45mm_HandSolder, symbol Device:C_Small
- added D10: 1N5819HW-FDICT, Diode_SMD:D_SOD-123, symbol Device:D_Schottky_Small_Filled
- J9: value Conn_01x12_Socket -> Solar in
Connections:
- net GND_Batt: now also C2.2
- net V_Solar_An: now also C2.1
- new net +Solar: D10.1 (K)
Other:
- moved on the sheet: D3, D4, D5, D6, D7, D8, D9, J9, R10

Commit message: update
Parts:
- added J7: Bench Power, Connector_JST:JST_PH_S2B-PH-K_1x02_P2.00mm_Horizontal, symbol Connector_Generic:Conn_01x02
Connections:
- net GND_Batt: now also J7.2 (Pin_2)
- net at D10.2 (A): now also J7.1 (Pin_1)
Changed lines of the file:
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@@
+	(wire
+		(pts
+			(xy 44.45 110.49) (xy 44.45 113.03)
+		)
+		(stroke
+			(width 0)
+			(type default)
+		)
+	)
 	(wire
 		(pts
@@
 		(pts
 			(xy 50.8 62.23) (xy 50.8 67.31)
+		)
+		(stroke
+			(width 0)
+			(type default)
+		)
+	)
+	(wire
+		(pts
+			(xy 41.91 110.49) (xy 44.45 110.49)
 		)
 		(stroke
@@
 	)
 	(symbol
+		(lib_id "Connector_Generic:Conn_01x02")
+		(at 36.83 107.95 0)
+		(mirror y)
+		(unit 1)
+		(exclude_from_sim no)
+		(in_bom yes)
+		(on_board yes)
+		(dnp no)
+		(property "Reference" "J7"
+			(at 36.83 116.84 0)
+			(effects
+				(font
+					(size 1.27 1.27)
+				)
+			)
+		)
+		(property "Value" "Bench Power"
+			(at 36.83 114.3 0)
+			(effects
+				(font
+					(size 1.27 1.27)
+				)
+			)
+		)
+		(property "Footprint" "Connector_JST:JST_PH_S2B-PH-K_1x02_P2.00mm_Horizontal"
+			(at 36.83 107.95 0)
+			(effects
+				(font
+					(size 1.27 1.27)
+				)
+				(hide yes)
+			)
+		)
+		(property "Datasheet" "~"
+			(at 36.83 107.95 0)
+			(effects
+				(font
+					(size 1.27 1.27)
+				)
+				(hide yes)
+			)
+		)
+		(property "Description" "Generic connector, single row, 01x02, script generated (kicad-library-utils/schlib/autogen/connector/)"
+			(at 36.83 107.95 0)
+			(effects
+				(font
+					(size 1.27 1.27)
+				)
+				(hide yes)
+			)
+		)
+		(pin "2"
+		)
+		(pin "1"
+		)
+		(instances
+			(project "Buoy PCB"
+				(path "/a041e2a6-7d41-458c-91f3-753821d3dfe9/e8f4d549-a7ac-4e6a-bad9-8d4daf54a22c"
+					(reference "J7")
+					(unit 1)
+				)
+			)
+		)
+	)
+	(symbol
 		(lib_id "power:GND")
 		(at 86.36 81.28 0)
@@
 					(unit 1)
 				)
+			)
+		)
+	)
+	(symbol
+		(lib_id "power:GND")
+		(at 44.45 113.03 0)
+		(unit 1)
+		(exclude_from_sim no)
+		(in_bom yes)
+		(on_board yes)
+		(dnp no)
+		(fields_autoplaced yes)
+		(property "Reference" "#PWR043"
+			(at 44.45 119.38 0)
+			(effects
+				(font
+					(size 1.27 1.27)
+				)
+				(hide yes)
+			)
+		)
+		(property "Value" "GND_Batt"
+			(at 44.45 118.11 0)
+			(effects
+				(font
+					(size 1.27 1.27)
+				)
+			)
+		)
+		(property "Footprint" ""
+			(at 44.45 113.03 0)
+			(effects
+				(font
+					(size 1.27 1.27)
+				)
+				(hide yes)
+			)
+		)
+		(property "Datasheet" ""
+			(at 44.45 113.03 0)
+			(effects
+				(font
+					(size 1.27 1.27)
+				)
+				(hide yes)
+			)
+		)
+		(property "Description" "Power symbol creates a global label with name \"GND\" , ground"
+			(at 44.45 113.03 0)
+			(effects
+				(font
+					(size 1.27 1.27)
+				)
+				(hide yes)
+			)
+		)
+		(pin "1"
+		)
+		(instances
+			(project "Buoy PCB"
+				(path "/a041e2a6-7d41-458c-91f3-753821d3dfe9/e8f4d549-a7ac-4e6a-bad9-8d4daf54a22c"
+					(reference "#PWR043")
+					(unit 1)
+				)

Commit message: changes adn updates
Parts:
- added C10, C9: 47μF, Capacitor_SMD:CP_Elec_5x5.9, symbol Device:C_Polarized_Small
- added C2: 100μF, Capacitor_SMD:CP_Elec_5x5.9, symbol Device:C_Polarized_Small
- added C3: 0.1μF, Capacitor_SMD:C_0805_2012Metric_Pad1.18x1.45mm_HandSolder, symbol Device:C_Small
- added C4: 10nF, Capacitor_SMD:C_0805_2012Metric_Pad1.18x1.45mm_HandSolder, symbol Device:C_Small
- added C5: 10pF, Capacitor_SMD:C_0805_2012Metric_Pad1.18x1.45mm_HandSolder, symbol Device:C_Small
- added C6: 1nF, Capacitor_SMD:C_0805_2012Metric_Pad1.18x1.45mm_HandSolder, symbol Device:C_Small
- added C7, C8: 0.1uF, Capacitor_SMD:C_0805_2012Metric_Pad1.18x1.45mm_HandSolder, symbol Device:C_Small
- added D11: SS34, Diode_SMD:D_SMA_Handsoldering, symbol Device:D_Schottky_Small_Filled
- added L1: 8.2uH, Inductor_SMD:L_Taiyo-Yuden_NR-60xx_HandSoldering, symbol Device:L_Small
- added R4: 29.4k, Resistor_SMD:R_0805_2012Metric_Pad1.20x1.40mm_HandSolder, symbol Device:R_Small
- added R5: 10k2, Resistor_SMD:R_0805_2012Metric_Pad1.20x1.40mm_HandSolder, symbol Device:R_Small
- added R6: 1k96, Resistor_SMD:R_0805_2012Metric_Pad1.20x1.40mm_HandSolder, symbol Device:R_Small
- added U1: TPS54331D, Package_SO:TI_SO-PowerPAD-8_ThermalVias, symbol Regulator_Switching:TPS54336ADDA
- J7: renamed from J9; footprint Connector_PinSocket_2.54mm:PinSocket_1x12_P2.54mm_Vertical -> Connector_JST:JST_PH_S12B-PH-K_1x12_P2.00mm_Horizontal; symbol Connector:Conn_01x12_Socket -> Connector_Generic:Conn_01x12
- R2: renamed from R8; value 10k -> 20k
- renumbered C2 to C1, J7 to J9, R10 to R1, R9 to R3
Connections:
- net +Solar_Batt is gone; now on net +Solar: D4.1 (K), D5.1 (K), D6.1 (K), D7.1 (K), D8.1 (K), D9.1 (K), R1.1, R2.1
- net +Solar: now also C2.1, C3.1, U1.2 (VIN)
- net GND_Batt renamed GND
- net GND: now also C10.2, C2.2, C3.2, C4.2, C5.1, C6.1, C8.1, C9.2, D11.2 (A), R6.2, U1.7 (GND), U1.9 (ETPAD)
- new net: R5.2, R6.1, U1.5 (VSENSE)
- new net: C6.2, R4.2
- new net: C5.2, R4.1, U1.6 (COMP)
- new net: C7.2, D11.1 (K), L1.1, U1.8 (PH)
- new net: C7.1, U1.1 (BOOT)
- new net: C4.1, U1.4 (SS)
- new net +5V: C10.1, C8.2, C9.1, L1.2, R5.1
- no-connect marks 0 -> 1
Other:
- moved on the sheet: C1, D10, D3, D4, D5, D6, D7, D8, D9, J9, R1, R2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

Commit message: .
Parts:
- added SW1: SW_SPDT, Button_Switch_THT:SW_Slide_SPDT_Angled_CK_OS102011MA1Q, symbol Switch:SW_SPDT
Connections:
- net +Solar: now also SW1.1 (A); no longer D4.1 (K), D5.1 (K), D6.1 (K), D7.1 (K), D8.1 (K), D9.1 (K)
- new net: D4.1 (K), D5.1 (K), D6.1 (K), D7.1 (K), D8.1 (K), D9.1 (K), SW1.2 (B)
- no-connect marks 1 -> 2
Changed lines of the file:
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@@
 		(at 162.56 85.09)
 	)
+	(no_connect
+		(at 102.87 85.09)
+	)
 	(wire
 		(pts
@@
 	(wire
 		(pts
-			(xy 129.54 82.55) (xy 162.56 82.55)
+			(xy 106.68 76.2) (xy 106.68 80.01)
 		)
 		(stroke
@@
 	(wire
 		(pts
-			(xy 80.01 80.01) (xy 80.01 82.55)
+			(xy 129.54 82.55) (xy 162.56 82.55)
 		)
 		(stroke
@@
 	(wire
 		(pts
+			(xy 106.68 80.01) (xy 102.87 80.01)
+		)
+		(stroke
+			(width 0)
+			(type default)
+		)
+	)
+	(wire
+		(pts
 			(xy 72.39 87.63) (xy 80.01 87.63)
 		)
@@
 	(wire
 		(pts
+			(xy 80.01 82.55) (xy 92.71 82.55)
+		)
+		(stroke
+			(width 0)
+			(type default)
+		)
+	)
+	(wire
+		(pts
 			(xy 64.77 90.17) (xy 64.77 95.25)
 		)
@@
 	)
 	(symbol
-		(lib_id "power:+BATT")
-		(at 80.01 80.01 0)
-		(unit 1)
-		(exclude_from_sim no)
-		(in_bom yes)
-		(on_board yes)
-		(dnp no)
-		(fields_autoplaced yes)
-		(property "Reference" "#PWR022"
-			(at 80.01 83.82 0)
-			(effects
-				(font
-					(size 1.27 1.27)
-				)
-				(hide yes)
-			)
-		)
-		(property "Value" "+Solar"
-			(at 80.01 74.93 0)
-			(effects
-				(font
-					(size 1.27 1.27)
-				)
-			)
-		)
-		(property "Footprint" ""
-			(at 80.01 80.01 0)
-			(effects
-				(font
-					(size 1.27 1.27)
-				)
-				(hide yes)
-			)
-		)
-		(property "Datasheet" ""
-			(at 80.01 80.01 0)
-			(effects
-				(font
-					(size 1.27 1.27)
-				)
-				(hide yes)
-			)
-		)
-		(property "Description" "Power symbol creates a global label with name \"+Solar\""
-			(at 80.01 80.01 0)
-			(effects
-				(font
-					(size 1.27 1.27)
-				)
-				(hide yes)
-			)
-		)
-		(pin "1"
-		)
-		(instances
-			(project "Buoy PCB"
-				(path "/a041e2a6-7d41-458c-91f3-753821d3dfe9/402c8c5f-ad4a-46d2-a42e-eba9c7fe5855/022691eb-6a52-45b1-ac3b-a806631f277d"
-					(reference "#PWR022")
-					(unit 1)
-				)
-			)
-		)
-	)
-	(symbol
 		(lib_id "power:GND")
 		(at 149.86 110.49 0)
@@
 	)
 	(symbol
+		(lib_id "Switch:SW_SPDT")
+		(at 97.79 82.55 0)
+		(unit 1)
+		(exclude_from_sim no)
+		(in_bom yes)
+		(on_board yes)
+		(dnp no)
+		(fields_autoplaced yes)
+		(property "Reference" "SW1"
+			(at 97.79 73.66 0)
+			(effects
+				(font
+					(size 1.27 1.27)
+				)
+			)
+		)
+		(property "Value" "SW_SPDT"
+			(at 97.79 76.2 0)
+			(effects
+				(font
+					(size 1.27 1.27)
+				)
+			)
+		)
+		(property "Footprint" "Button_Switch_THT:SW_Slide_SPDT_Angled_CK_OS102011MA1Q"
+			(at 97.79 82.55 0)
+			(effects
+				(font
+					(size 1.27 1.27)
+				)
+				(hide yes)
+			)
+		)
+		(property "Datasheet" "~"
+			(at 97.79 90.17 0)
+			(effects
+				(font
+					(size 1.27 1.27)
+				)
+				(hide yes)
+			)
+		)
+		(property "Description" "Switch, single pole double throw"
+			(at 97.79 82.55 0)
+			(effects
+				(font
+					(size 1.27 1.27)
+				)
+				(hide yes)
+			)
+		)
+		(pin "1"
+		)
+		(pin "2"
+		)
+		(pin "3"
+		)
+		(instances
+			(project "Buoy PCB"
+				(path "/a041e2a6-7d41-458c-91f3-753821d3dfe9/402c8c5f-ad4a-46d2-a42e-eba9c7fe5855/022691eb-6a52-45b1-ac3b-a806631f277d"
+					(reference "SW1")
+					(unit 1)
+				)
+			)
+		)
+	)
+	(symbol
 		(lib_id "power:GND")
 		(at 198.12 110.49 0)
@@
 					(unit 1)
 				)
+			)
+		)
+	)
+	(symbol
+		(lib_id "power:+BATT")
+		(at 106.68 76.2 0)
+		(unit 1)
+		(exclude_from_sim no)
+		(in_bom yes)
+		(on_board yes)
+		(dnp no)
+		(fields_autoplaced yes)
+		(property "Reference" "#PWR06"
+			(at 106.68 80.01 0)
+			(effects
+				(font
+					(size 1.27 1.27)
+				)
+				(hide yes)
+			)
+		)
+		(property "Value" "+Solar"
+			(at 106.68 71.12 0)
+			(effects
+				(font
+					(size 1.27 1.27)
+				)
+			)
+		)
+		(property "Footprint" ""
+			(at 106.68 76.2 0)
+			(effects
+				(font
+					(size 1.27 1.27)
+				)
+				(hide yes)
+			)
+		)
+		(property "Datasheet" ""
+			(at 106.68 76.2 0)
+			(effects
+				(font
+					(size 1.27 1.27)
+				)
+				(hide yes)
+			)
+		)
+		(property "Description" "Power symbol creates a global label with name \"+Solar\""
+			(at 106.68 76.2 0)
+			(effects
+				(font
+					(size 1.27 1.27)
+				)
+				(hide yes)
+			)
+		)
+		(pin "1"
+		)
+		(instances
+			(project "Buoy PCB"
+				(path "/a041e2a6-7d41-458c-91f3-753821d3dfe9/402c8c5f-ad4a-46d2-a42e-eba9c7fe5855/022691eb-6a52-45b1-ac3b-a806631f277d"
+					(reference "#PWR06")
+					(unit 1)
+				)
