File: Main PCB KiCAD/solar.kicad_sch (KiCad schematic)
At the start: 30 parts, among them J7 Solar in, J9 Bench Power, SW1 SW_SPDT, U1 TPS54331D

Commit message: .
Connections:
- net GND: no longer C2.2, C3.2, D3.1 (K), J7.10 (Pin_10), J7.12 (Pin_12), J7.2 (Pin_2), J7.4 (Pin_4), J7.6 (Pin_6), J7.8 (Pin_8), J9.2 (Pin_2)
- new net Front PCB GND: C2.2, C3.2, D3.1 (K), J7.10 (Pin_10), J7.12 (Pin_12), J7.2 (Pin_2), J7.4 (Pin_4), J7.6 (Pin_6), J7.8 (Pin_8), J9.2 (Pin_2)

Commit message: .
Parts:
- removed D10: 1N5819HW-FDICT, Diode_SMD:D_SOD-123, symbol Device:D_Schottky_Small_Filled
- removed J9: Bench Power, Connector_JST:JST_PH_S2B-PH-K_1x02_P2.00mm_Horizontal, symbol Connector_Generic:Conn_01x02
- J7: footprint Connector_JST:JST_PH_S12B-PH-K_1x12_P2.00mm_Horizontal -> Connector_JST:JST_EH_S12B-EH_1x12_P2.50mm_Horizontal
Connections:
- net Front PCB GND is gone; now on net GND: C2.2, C3.2, D3.1 (K), J7.10 (Pin_10), J7.12 (Pin_12), J7.2 (Pin_2), J7.4 (Pin_4), J7.6 (Pin_6), J7.8 (Pin_8)
- net +5V: now also SW1.1 (A); no longer C10.1, C8.2, C9.1, L1.2, R5.1
- net +Solar: now also D4.1 (K), D5.1 (K), D6.1 (K), D7.1 (K), D8.1 (K), D9.1 (K); no longer SW1.1 (A)
- new net: C10.1, C8.2, C9.1, L1.2, R5.1, SW1.2 (B)
- no-connect marks 2 -> 1
Other:
- moved on the sheet: SW1

Commit message: .
Parts:
- removed C10, C9: 47μF, Capacitor_SMD:CP_Elec_5x5.9, symbol Device:C_Polarized_Small
- removed C4: 10nF, Capacitor_SMD:C_0805_2012Metric_Pad1.18x1.45mm_HandSolder, symbol Device:C_Small
- removed C5: 10pF, Capacitor_SMD:C_0805_2012Metric_Pad1.18x1.45mm_HandSolder, symbol Device:C_Small
- removed C6: 1nF, Capacitor_SMD:C_0805_2012Metric_Pad1.18x1.45mm_HandSolder, symbol Device:C_Small
- removed C7, C8: 0.1uF, Capacitor_SMD:C_0805_2012Metric_Pad1.18x1.45mm_HandSolder, symbol Device:C_Small
- removed D11: SS34, Diode_SMD:D_SMA_Handsoldering, symbol Device:D_Schottky_Small_Filled
- removed L1: 8.2uH, Inductor_SMD:L_Taiyo-Yuden_NR-60xx_HandSoldering, symbol Device:L_Small
- removed R4: 29.4k, Resistor_SMD:R_0805_2012Metric_Pad1.20x1.40mm_HandSolder, symbol Device:R_Small
- removed R5: 10k2, Resistor_SMD:R_0805_2012Metric_Pad1.20x1.40mm_HandSolder, symbol Device:R_Small
- removed R6: 1k96, Resistor_SMD:R_0805_2012Metric_Pad1.20x1.40mm_HandSolder, symbol Device:R_Small
- removed U1: TPS54331D, Package_SO:TI_SO-PowerPAD-8_ThermalVias, symbol Regulator_Switching:TPS54336ADDA
Connections:
- no-connect marks 1 -> 0
Other:
- note added: "5V regulator needed (1 A)"
- moved on the sheet: C2, C3
