File: Main PCB KiCAD/Shrimp.kicad_sch (KiCad schematic)
At the start: 4 parts, among them J10 P3, J13 P2, J14 P4, J15 P5

Commit message: changes adn updates
Parts:
- renumbered J13 to J10, J14 to J11, J10 to J12, J15 to J13
Connections:
- net +5V renamed Front PCB +5V
- net 10 | LoRa MOSI renamed MOSI
- net 11 | LoRa MISO renamed MISO
- net 15 | 32K XP renamed GPIO_15  / ADC2_CH4
- net 16 | 32K XN renamed GPIO_16  / ADC2_CH5
- net 18 | LED renamed GPIO_18  / HeartBeat_LED
- net GND renamed Front PCB GND
- net GPIO_17  /ADC2_CH6 renamed GPIO_17  / ADC2_CH6
- net GPIO_45 renamed I2C_SCL
- net GPIO_46 renamed I2C_SDA
Other:
- note added: "https://github.com/jhiggason/lorawirelesstracker"
- note added: "https://randomnerdtutorials.com/esp32-i2c-communication-arduino-ide/"
