File: Main PCB KiCAD/Buoy PCB.kicad_pcb (KiCad board)
At the start: 2 copper layers, 219.2 x 111.7 mm, 73 parts, among them J1 Conn_01x12_Socket, J10 USB_B_Micro, J11 Battery 1, J12 Battery 2, J2 Conn_01x12_Socket, J3 Conn_01x12_Pin, J4 Conn_01x12_Pin, J5 UART, J6 ICSP, J7 I2C, J8 RS485, J9 Conn_01x12_Socket, Q1 Q_NMOS_DSG, Q2 Q_NMOS_DSG, U1 ATmega328P-P, U2 MAX3072E, U4 MCP73834T-FCI/UN, Y1 16 MHz

Commit message: cleanup
Parts:
- removed C4: 100nF, Capacitor_SMD:C_0805_2012Metric_Pad1.18x1.45mm_HandSolder
- removed C5, C6: 22pF, Capacitor_SMD:C_0805_2012Metric_Pad1.18x1.45mm_HandSolder
- removed J10: USB_B_Micro, Connector_USB:USB_Micro-B_Amphenol_10103594-0001LF_Horizontal
- removed J5: UART, Connector_PinHeader_2.54mm:PinHeader_1x05_P2.54mm_Vertical
- removed J6: ICSP, Connector_PinHeader_2.54mm:PinHeader_2x03_P2.54mm_Vertical
- removed J7: I2C, Connector_PinHeader_2.54mm:PinHeader_1x04_P2.54mm_Vertical
- removed R1, R2, R6: 10k, Resistor_SMD:R_0805_2012Metric_Pad1.20x1.40mm_HandSolder
- removed R3, R4: 1k, Resistor_SMD:R_0805_2012Metric_Pad1.20x1.40mm_HandSolder
- removed R5: 1M, Resistor_SMD:R_0805_2012Metric_Pad1.20x1.40mm_HandSolder
- removed TP1: HB, TestPoint:TestPoint_Pad_D1.0mm
- removed TP2: 5V, TestPoint:TestPoint_Pad_D1.0mm
- removed TP3: GND, TestPoint:TestPoint_Pad_D1.0mm
- removed U1: ATmega328P-P, Package_DIP:DIP-28_W7.62mm
- removed Y1: 16 MHz, Crystal:Crystal_SMD_EuroQuartz_MQ-4Pin_7.0x5.0mm_HandSoldering
- added A1: RaspberryPi_Pico_W, Module:RaspberryPi_Pico_Common_Unspecified, F.Cu at (78.5, 62.7)
- added D18: WS2812B, LED_SMD:LED_WS2812B_PLCC4_5.0x5.0mm_P3.2mm, F.Cu at (266.2, 54.4)
- added D19: WS2812B, LED_SMD:LED_WS2812B_PLCC4_5.0x5.0mm_P3.2mm, F.Cu at (259.6, 37.1)
- C1, C3: value 100nF -> 1u
- C2: value 10uF -> 1u; footprint Capacitor_SMD:C_Elec_6.3x5.8 -> Capacitor_SMD:C_0805_2012Metric_Pad1.18x1.45mm_HandSolder
- D1: value Red -> WS2812B; footprint Diode_SMD:D_0805_2012Metric_Pad1.15x1.40mm_HandSolder -> LED_SMD:LED_WS2812B_PLCC4_5.0x5.0mm_P3.2mm
- D2: value Green -> WS2812B; footprint Diode_SMD:D_0805_2012Metric_Pad1.15x1.40mm_HandSolder -> LED_SMD:LED_WS2812B_PLCC4_5.0x5.0mm_P3.2mm
- J1: value Conn_01x12_Socket -> Top B; moved to B.Cu
- J12: moved to B.Cu
- J2: value Conn_01x12_Socket -> Top A; moved to B.Cu
- J3: value Conn_01x12_Pin -> Bottom B
- J4: value Conn_01x12_Pin -> Bottom A
- J9: value Conn_01x12_Socket -> Solar in
- U4: footprint Package_SO:SOIC-8_3.9x4.9mm_P1.27mm -> Silicon-Standard:MSOP-10-GNDPAD
- moved JP2 249.3 mm to (-15.3, 138.7)
- moved U2 249.3 mm to (-13.3, 133.7)
- moved R7 248.0 mm to (-14.0, 126.0), turned to 0 degrees
- moved D2 187.9 mm to (256.5, 67.6)
- moved D10 179.0 mm to (61.2, 82.5), turned to -90 degrees
- moved D11 153.5 mm to (88.4, 82.3), turned to 90 degrees
- moved JP3 152.5 mm to (95.5, 78.2), turned to -90 degrees
- moved J12 149.9 mm to (26.2, 106.6), turned to 0 degrees
- moved D9 146.4 mm to (76.5, 82.5)
- moved R12 141.4 mm to (82.3, 78.2), turned to 90 degrees
- moved R14 134.1 mm to (88.4, 78.2)
- moved D13 129.9 mm to (92.5, 82.3), turned to 90 degrees
- moved J11 127.5 mm to (36.1, 106.1), turned to 0 degrees
- moved JP1 127.0 mm to (-19.5, 126.3)
- moved R13 126.5 mm to (98.6, 86.4), turned to 180 degrees
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Connections:
- C1 pad 1: +5V -> /V_Batt_An
- C1 pad 2: GND -> -Batt
- C2 pad 1: +5V -> /V_Solar_An
- C3 pad 1: Net-(U1-AREF) -> +Solar
- C7 pad 1: +Solar_Batt -> +Solar
- C7 pad 2: GND_Batt -> GND
- C9 pad 1: +3.3V_bat -> +3.3V
- D1 pad 1: GND -> +5V
- D1 pad 2: Net-(D1-A) -> Net-(D1-DOUT)
- D10 pad 2: Net-(D10-A) -> unconnected-(D10-A-Pad2)
- D11 pad 1: Net-(D11-K) -> /Battery Charger/Status1
- D12 pad 1: Net-(D12-K) -> /Battery Charger/Status2
- D12 pad 2: Net-(D11-A) -> Net-(D12-A)
- D13 pad 1: Net-(D13-K) -> /Battery Charger/PG
- D13 pad 2: Net-(D11-A) -> Net-(D13-A)
- D14 pad 4: unconnected-(D14-DIN-Pad4) -> /Arduino Mega/NeoPixle_Out
- D17 pad 2: unconnected-(D17-DOUT-Pad2) -> Net-(D1-DIN)
- D2 pad 1: GND -> +5V
- D3 pad 1: GND_Batt -> GND
- D4 pad 1: +Solar_Batt -> +Solar
- D5 pad 1: +Solar_Batt -> +Solar
- D6 pad 1: +Solar_Batt -> +Solar
- D7 pad 1: +Solar_Batt -> +Solar
- D8 pad 1: +Solar_Batt -> +Solar
- D9 pad 1: +Solar_Batt -> +Solar
- J1 pad 1: +3.3V -> unconnected-(J1-Pin_1-Pad1)
- J1 pad 2: +Solar -> unconnected-(J1-Pin_2-Pad2)
- J1 pad 3: GND -> unconnected-(J1-Pin_3-Pad3)
- J1 pad 4: GND -> unconnected-(J1-Pin_4-Pad4)
- J1 pad 7: GND -> unconnected-(J1-Pin_7-Pad7)
- J2 pad 12: GND -> unconnected-(J2-Pin_12-Pad12)
- J3 pad 1: +3.3V_bat -> unconnected-(J3-Pin_1-Pad1)
- J3 pad 2: +Solar_Batt -> unconnected-(J3-Pin_2-Pad2)
- J3 pad 3: GND_Batt -> unconnected-(J3-Pin_3-Pad3)
- J3 pad 4: GND_Batt -> unconnected-(J3-Pin_4-Pad4)
- J3 pad 5: /V_Batt_An -> unconnected-(J3-Pin_5-Pad5)
- J3 pad 6: /V_Solar_An -> unconnected-(J3-Pin_6-Pad6)
- J3 pad 7: GND_Batt -> unconnected-(J3-Pin_7-Pad7)
- J4 pad 12: GND_Batt -> unconnected-(J4-Pin_12-Pad12)
- J9 pad 10: GND_Batt -> GND
- J9 pad 12: GND_Batt -> GND
- J9 pad 2: GND_Batt -> GND
- J9 pad 4: GND_Batt -> GND
- J9 pad 6: GND_Batt -> GND
- J9 pad 8: GND_Batt -> GND
- JP3 pad 1: Net-(D11-A) -> Net-(JP3-A)
- JP3 pad 2: +Solar_Batt -> +Solar
- Q2 pad 2: GND_Batt -> GND
- R10 pad 1: +Solar_Batt -> +Solar
- R14 pad 1: Net-(D11-K) -> Net-(JP3-A)
- R14 pad 2: /Battery Charger/Status1 -> Net-(D11-A)
- R15 pad 1: Net-(D12-K) -> Net-(JP3-A)
- R15 pad 2: /Battery Charger/Status2 -> Net-(D12-A)
- R16 pad 1: Net-(D13-K) -> Net-(JP3-A)
- R16 pad 2: /Battery Charger/PG -> Net-(D13-A)
- R17 pad 1: +3.3V_bat -> +3.3V
- R18 pad 1: +3.3V_bat -> +3.3V
- R19 pad 1: +3.3V_bat -> +3.3V
- R21 pad 2: GND_Batt -> GND
- R8 pad 1: +Solar_Batt -> +Solar
- R9 pad 2: GND_Batt -> GND
- U4 pad 1: +Solar_Batt -> +Solar
- U4 pad 2: +Solar_Batt -> +Solar
Routing:
- net +5V: track 0.00 -> 136.6 mm
- net Net-(D1-DOUT): track 0.00 -> 23.3 mm
- net Net-(D18-DIN): track 0.00 -> 22.5 mm
- net Net-(D18-DOUT): track 0.00 -> 22.1 mm
- net Net-(D1-DIN): track 0.00 -> 21.6 mm
- net +Solar: track 38.6 -> 58.1 mm, vias 0 -> 2
- net Net-(D16-DOUT): track 0.00 -> 18.4 mm
- net Net-(D14-DOUT): track 0.00 -> 16.0 mm
- net +Solar_Batt: track 14.8 -> 0.00 mm
- net Net-(D1-A): track 13.7 -> 0.00 mm
- net +Batt: track 13.3 -> 26.1 mm, vias 0 -> 2
- net /Battery Charger/PG: track 0.00 -> 12.7 mm, vias 0 -> 2
- net /V_Solar_An: track 1.81 -> 14.1 mm
- net Net-(D15-DOUT): track 0.00 -> 11.6 mm
- net /V_Batt_An: track 0.00 -> 11.6 mm
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- added copper zone on B.Cu, net +3.3V
- added copper zone on F.Cu, net unconnected-(J3-Pin_3-Pad3)
- removed copper zone on F.Cu, net GND_Batt

Commit message: update
Parts:
- added J5: Top Interface, Connector_PinSocket_2.54mm:PinSocket_1x12_P2.54mm_Vertical, B.Cu at (255.3, 48.5)
- added J6: Top, Connector_PinHeader_2.54mm:PinHeader_1x12_P2.54mm_Horizontal, F.Cu at (67.6, 37.7)
- added J7: Bench Power, Connector_JST:JST_PH_S2B-PH-K_1x02_P2.00mm_Horizontal, F.Cu at (58.8, 40.7)
- J1: value Top B -> Front B
- J2: value Top A -> Front A
- J3: value Bottom B -> Back B
- J4: value Bottom A -> Back A
Connections:
- D1 pad 1: +5V -> Top PCB +5V
- D1 pad 3: GND -> Top PCB GND
- D10 pad 2: unconnected-(D10-A-Pad2) -> Net-(D10-A)
- D14 pad 1: +5V -> Top PCB +5V
- D14 pad 3: GND -> Top PCB GND
- D14 pad 4: /Arduino Mega/NeoPixle_Out -> /Top PCB/NeoPixle_In
- D15 pad 1: +5V -> Top PCB +5V
- D15 pad 3: GND -> Top PCB GND
- D16 pad 1: +5V -> Top PCB +5V
- D16 pad 3: GND -> Top PCB GND
- D17 pad 1: +5V -> Top PCB +5V
- D17 pad 3: GND -> Top PCB GND
- D18 pad 1: +5V -> Top PCB +5V
- D18 pad 3: GND -> Top PCB GND
- D19 pad 1: +5V -> Top PCB +5V
- D19 pad 3: GND -> Top PCB GND
- D2 pad 1: +5V -> Top PCB +5V
- D2 pad 3: GND -> Top PCB GND
Routing:
- net +5V: track 136.6 -> 0.00 mm
- net /Top PCB/NeoPixle_In: track 0.00 -> 29.0 mm
- net Net-(D16-DOUT): track 18.4 -> 20.6 mm
- net Net-(D14-DOUT): track 16.0 -> 15.3 mm
- net Top PCB GND: track 0.00 -> 0.52 mm, vias 0 -> 8
- added copper zone on F.Cu, net Top PCB +5V
- added copper zone on B.Cu, net Top PCB GND
- removed copper zone on B.Cu, net GND

Commit message: updates
Parts:
- removed A1: RaspberryPi_Pico_W, Module:RaspberryPi_Pico_Common_Unspecified
- added J10: P3, Connector_PinSocket_2.54mm:PinSocket_1x08_P2.54mm_Vertical, F.Cu at (-131.1, 108.0)
- added J13: P2, Connector_PinSocket_2.54mm:PinSocket_1x08_P2.54mm_Vertical, F.Cu at (-126.5, 108.0)
- added J14: P4, Connector_PinHeader_2.54mm:PinHeader_1x16_P2.54mm_Vertical, F.Cu at (-140.3, 108.0)
- added J15: P5, Connector_PinHeader_2.54mm:PinHeader_1x16_P2.54mm_Vertical, F.Cu at (-135.7, 108.0)

Commit message: changes adn updates
Parts:
- removed C11: 100nF, Capacitor_SMD:C_0805_2012Metric_Pad1.18x1.45mm_HandSolder
- removed D13: RED, LED_SMD:LED_0805_2012Metric_Pad1.15x1.40mm_HandSolder
- removed J14: P4, Connector_PinHeader_2.54mm:PinHeader_1x16_P2.54mm_Vertical
- removed J15: P5, Connector_PinHeader_2.54mm:PinHeader_1x16_P2.54mm_Vertical
- removed JP3: LEDs, Jumper:SolderJumper-2_P1.3mm_Bridged_RoundedPad1.0x1.5mm
- removed Q1, Q2: Q_NMOS_DSG, Package_TO_SOT_SMD:SOT-23
- removed R10, R13: 1k, Resistor_SMD:R_0805_2012Metric_Pad1.20x1.40mm_HandSolder
- removed R11, R12, R9: 10k, Resistor_SMD:R_0805_2012Metric_Pad1.20x1.40mm_HandSolder
- removed R14, R15, R16, R20: 330, Resistor_SMD:R_0805_2012Metric_Pad1.20x1.40mm_HandSolder
- removed R17, R18, R19: 22k, Resistor_SMD:R_0805_2012Metric_Pad1.20x1.40mm_HandSolder
- removed R21: 2.7k, Resistor_SMD:R_0805_2012Metric_Pad1.20x1.40mm_HandSolder
- removed U4: MCP73834T-FCI/UN, Silicon-Standard:MSOP-10-GNDPAD
- added C4: 10nF, Capacitor_SMD:C_0805_2012Metric_Pad1.18x1.45mm_HandSolder, F.Cu at (62.2, 78.1)
- added C5: 10pF, Capacitor_SMD:C_0805_2012Metric_Pad1.18x1.45mm_HandSolder, F.Cu at (65.4, 89.5)
- added C6: 1nF, Capacitor_SMD:C_0805_2012Metric_Pad1.18x1.45mm_HandSolder, F.Cu at (60.3, 87.0)
- added L1: 8.2uH, Inductor_SMD:L_Taiyo-Yuden_NR-60xx_HandSoldering, F.Cu at (65.4, 95.2)
- added R1: 1k, Resistor_SMD:R_0805_2012Metric_Pad1.20x1.40mm_HandSolder, F.Cu at (59.7, 40.6)
- added R2: 20k, Resistor_SMD:R_0805_2012Metric_Pad1.20x1.40mm_HandSolder, F.Cu at (38.5, 108.8)
- added R3: 10k, Resistor_SMD:R_0805_2012Metric_Pad1.20x1.40mm_HandSolder, F.Cu at (38.5, 111.8)
- added R4: 29.4k, Resistor_SMD:R_0805_2012Metric_Pad1.20x1.40mm_HandSolder, F.Cu at (60.3, 89.5)
- added R5: 10k2, Resistor_SMD:R_0805_2012Metric_Pad1.20x1.40mm_HandSolder, F.Cu at (59.7, 91.7)
- added R6: 1k96, Resistor_SMD:R_0805_2012Metric_Pad1.20x1.40mm_HandSolder, F.Cu at (59.7, 94.0)
- added U1: TPS54331D, Package_SO:TI_SO-PowerPAD-8_ThermalVias, F.Cu at (65.3, 84.4)
- C10: value 1uF -> 47μF; footprint Capacitor_SMD:C_0805_2012Metric_Pad1.18x1.45mm_HandSolder -> Capacitor_SMD:CP_Elec_5x5.9
- C2: value 1u -> 100μF; footprint Capacitor_SMD:C_0805_2012Metric_Pad1.18x1.45mm_HandSolder -> Capacitor_SMD:CP_Elec_5x5.9
- C3: value 1u -> 0.1μF
- C7, C8: value 1u -> 0.1uF
- C9: value 1u -> 47μF; footprint Capacitor_SMD:C_0805_2012Metric_Pad1.18x1.45mm_HandSolder -> Capacitor_SMD:CP_Elec_5x5.9
- D11: value RED -> SS34; footprint LED_SMD:LED_0805_2012Metric_Pad1.15x1.40mm_HandSolder -> Diode_SMD:D_SMA_Handsoldering
- J10: value P3 -> P2
- J11: value Battery 1 -> P4; footprint Connector_JST:JST_PH_S2B-PH-K_1x02_P2.00mm_Horizontal -> Connector_PinSocket_2.54mm:PinSocket_1x16_P2.54mm_Vertical; moved to F.Cu
- J12: value Battery 2 -> P3; footprint Connector_JST:JST_PH_S2B-PH-K_1x02_P2.00mm_Horizontal -> Connector_PinSocket_2.54mm:PinSocket_1x08_P2.54mm_Vertical; moved to F.Cu
- J13: value P2 -> P5; footprint Connector_PinSocket_2.54mm:PinSocket_1x08_P2.54mm_Vertical -> Connector_PinSocket_2.54mm:PinSocket_1x16_P2.54mm_Vertical
- J7: value Bench Power -> Solar in; footprint Connector_JST:JST_PH_S2B-PH-K_1x02_P2.00mm_Horizontal -> Connector_JST:JST_PH_S12B-PH-K_1x12_P2.00mm_Horizontal
- J8: footprint Connector_Molex:Molex_Nano-Fit_105309-xx08_1x08_P2.50mm_Vertical -> Connector_JST:JST_PH_S8B-PH-K_1x08_P2.00mm_Horizontal
- J9: value Solar in -> Bench Power; footprint Connector_PinSocket_2.54mm:PinSocket_1x12_P2.54mm_Vertical -> Connector_JST:JST_PH_S2B-PH-K_1x02_P2.00mm_Horizontal
- R8: value 10k -> 1k
- moved J13 223.7 mm to (94.0, 70.5)
- moved J10 211.1 mm to (71.1, 47.6)
- moved J8 99.7 mm to (105.5, 58.5), turned to 90 degrees
- moved J12 89.9 mm to (94.0, 47.6)
- moved C1 58.3 mm to (23.6, 92.2), turned to 0 degrees
- moved D12 56.0 mm to (55.2, 38.7), turned to 0 degrees
- moved D3 52.0 mm to (55.2, 40.6), turned to 0 degrees
- moved C10 50.4 mm to (64.8, 111.8), turned to 180 degrees
- moved U2 50.3 mm to (36.9, 129.5)
- moved JP1 50.3 mm to (30.6, 122.1)
- moved JP2 50.3 mm to (34.8, 134.5)
- moved R7 50.3 mm to (36.2, 121.8)
- moved J11 49.9 mm to (71.1, 70.5)
- moved J9 48.6 mm to (58.8, 44.4), turned to -90 degrees
- moved R8 46.6 mm to (59.7, 38.7), turned to 180 degrees
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Connections:
- C1 pad 1: /V_Batt_An -> /Front PCB/V_Solar_An
- C1 pad 2: -Batt -> GND
- C10 pad 1: +Batt -> +5V
- C10 pad 2: -Batt -> GND
- C2 pad 1: /V_Solar_An -> +Solar
- C7 pad 1: +Solar -> Net-(U1-BOOT)
- C7 pad 2: GND -> Net-(D11-K)
- C8 pad 1: +Batt -> GND
- C8 pad 2: GND -> +5V
- C9 pad 1: +3.3V -> +5V
- D11 pad 1: /Battery Charger/Status1 -> Net-(D11-K)
- D11 pad 2: Net-(D11-A) -> GND
- D12 pad 1: /Battery Charger/Status2 -> GND
- J1 pad 1: unconnected-(J1-Pin_1-Pad1) -> Front PCB +5V
- J1 pad 2: unconnected-(J1-Pin_2-Pad2) -> Front PCB GND
- J1 pad 3: unconnected-(J1-Pin_3-Pad3) -> Front PCB +5V
- J1 pad 4: unconnected-(J1-Pin_4-Pad4) -> Front PCB GND
- J10 pad 1: unconnected-(J10-Pin_1-Pad1) -> Front PCB +5V
- J10 pad 2: unconnected-(J10-Pin_2-Pad2) -> Front PCB GND
- J10 pad 3: unconnected-(J10-Pin_3-Pad3) -> +3V3
- J10 pad 4: unconnected-(J10-Pin_4-Pad4) -> Front PCB GND
- J10 pad 5: unconnected-(J10-Pin_5-Pad5) -> +3V3
- J10 pad 6: unconnected-(J10-Pin_6-Pad6) -> Front PCB GND
- J10 pad 7: unconnected-(J10-Pin_7-Pad7) -> Vext
- J10 pad 8: unconnected-(J10-Pin_8-Pad8) -> Front PCB GND
- J11 pad 1: +Batt -> /Front PCB/Shrimp/RESET_SW | CHIP_PU
- J11 pad 2: -Batt -> /Front PCB/Shrimp/USER_SW | 0
- J12 pad 1: +Batt -> /Front PCB/Heart Beat
- J12 pad 2: -Batt -> /Front PCB/Shrimp/17
- J13 pad 1: unconnected-(J13-Pin_1-Pad1) -> /Front PCB/Shrimp/46
- J13 pad 2: unconnected-(J13-Pin_2-Pad2) -> /Front PCB/Shrimp/45
- J13 pad 3: unconnected-(J13-Pin_3-Pad3) -> /Front PCB/Shrimp/44 | U0RXD
- J13 pad 4: unconnected-(J13-Pin_4-Pad4) -> /Front PCB/Shrimp/43 | U0TXD
- J13 pad 5: unconnected-(J13-Pin_5-Pad5) -> /Front PCB/Shrimp/14 | DIO1
- J13 pad 6: unconnected-(J13-Pin_6-Pad6) -> /Front PCB/Shrimp/13 | LoRa Busy
- J13 pad 7: unconnected-(J13-Pin_7-Pad7) -> /Front PCB/Shrimp/12 | LoRa RST
- J13 pad 8: unconnected-(J13-Pin_8-Pad8) -> /Front PCB/Shrimp/11 | LoRa MISO
- J2 pad 1: unconnected-(J2-Pin_1-Pad1) -> Front PCB +5V
- J2 pad 2: unconnected-(J2-Pin_2-Pad2) -> Front PCB GND
- J2 pad 3: unconnected-(J2-Pin_3-Pad3) -> Front PCB +5V
- J2 pad 4: unconnected-(J2-Pin_4-Pad4) -> Front PCB GND
- J3 pad 1: unconnected-(J3-Pin_1-Pad1) -> Back PCB +5V
- J3 pad 2: unconnected-(J3-Pin_2-Pad2) -> Back PCB GND
- J3 pad 3: unconnected-(J3-Pin_3-Pad3) -> Back PCB +5V
- J3 pad 4: unconnected-(J3-Pin_4-Pad4) -> Back PCB GND
- J4 pad 1: unconnected-(J4-Pin_1-Pad1) -> Back PCB +5V
- J4 pad 2: unconnected-(J4-Pin_2-Pad2) -> Back PCB GND
- J4 pad 3: unconnected-(J4-Pin_3-Pad3) -> Back PCB +5V
- J4 pad 4: unconnected-(J4-Pin_4-Pad4) -> Back PCB GND
- J6 pad 10: unconnected-(J6-Pin_10-Pad10) -> Front PCB +5V
- J6 pad 11: unconnected-(J6-Pin_11-Pad11) -> Front PCB GND
- J6 pad 12: unconnected-(J6-Pin_12-Pad12) -> /Front PCB/Shrimp/37
- J6 pad 9: unconnected-(J6-Pin_9-Pad9) -> Front PCB GND
- J7 pad 1: Net-(D10-A) -> Net-(D4-A)
- J9 pad 1: Net-(D4-A) -> Net-(D10-A)
- R8 pad 1: +Solar -> /Front PCB/Heart Beat
- R8 pad 2: /V_Solar_An -> Net-(D12-A)
Routing:
- net /Front PCB/Heart Beat: track 0.00 -> 37.7 mm
- net +Batt: track 26.1 -> 0.00 mm, vias 2 -> 0
- net Net-(D11-K): track 0.00 -> 25.7 mm
- net -Batt: track 25.5 -> 0.00 mm, vias 2 -> 0
- net +5V: track 0.00 -> 23.0 mm, vias 0 -> 2
- net /V_Solar_An: track 14.1 -> 0.00 mm
- net /Battery Charger/PG: track 12.7 -> 0.00 mm, vias 2 -> 0
- net +Solar: track 58.1 -> 45.8 mm, vias 2 -> 0
- net /V_Batt_An: track 11.6 -> 0.00 mm
- net /Battery Charger/Status1: track 10.8 -> 0.00 mm
- net Net-(U1-VSENSE): track 0.00 -> 10.5 mm
- net /Battery Charger/Status2: track 9.61 -> 0.00 mm
- net Net-(D9-A): track 0.00 -> 8.55 mm
- net Net-(D8-A): track 0.00 -> 7.09 mm
- net Net-(JP3-A): track 6.75 -> 0.00 mm
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- added copper zone on F.Cu, net Back PCB +5V
- added copper zone on F.Cu, net Front PCB +5V
- added copper zone on B.Cu, net Front PCB GND
- removed copper zone on B.Cu, net +3.3V
- removed copper zone on F.Cu, net GND
- removed copper zone on F.Cu, net unconnected-(J3-Pin_3-Pad3)
Other:
- board size 219.2 x 111.7 mm -> 191.8 x 100 mm

Commit message: Update Buoy PCB.kicad_pcb
Parts:
- moved D15 0.79 mm to (201.9, 53.3), turned to 50 degrees
Routing:
- net Net-(D14-DOUT): track 15.3 -> 17.9 mm
- net Top PCB GND: track 0.52 -> 3.03 mm
- net Net-(D15-DOUT): track 11.6 -> 10.3 mm
Changed lines of the file:
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@@
 	(footprint "LED_SMD:LED_WS2812B_PLCC4_5.0x5.0mm_P3.2mm"
 		(layer "F.Cu")
-		(at 202.221 52.607)
+		(at 201.93 53.34 50)
 		(descr "5.0mm x 5.0mm Addressable RGB LED NeoPixel, https://cdn-shop.adafruit.com/datasheets/WS2812B.pdf")
 		(tags "LED RGB NeoPixel PLCC-4 5050")
 		(property "Reference" "D15"
-			(at 0 -3.5 0)
+			(at -0.000001 -3.5 50)
 			(layer "F.SilkS")
 			(effects
@@
 		)
 		(property "Value" "WS2812B"
-			(at 0 4 0)
+			(at 0 4 50)
 			(layer "F.Fab")
 			(effects
@@
 		)
 		(property "Datasheet" "https://cdn-shop.adafruit.com/datasheets/WS2812B.pdf"
-			(at 0 0 0)
+			(at 0 0 50)
 			(unlocked yes)
 			(layer "F.Fab")
@@
 		)
 		(property "Description" "RGB LED with integrated controller"
-			(at 0 0 0)
+			(at 0 0 50)
 			(unlocked yes)
 			(layer "F.Fab")
@@
 		(attr smd)
 		(fp_line
-			(start -3.5 -2.75)
-			(end -3.5 2.75)
+			(start -3.5 -2.749999)
+			(end -3.499999 2.75)
 			(stroke
 				(width 0.12)
@@
 		)
 		(fp_line
-			(start -3.5 -2.75)
-			(end 3.5 -2.75)
+			(start -3.5 -2.749999)
+			(end 3.499999 -2.75)
 			(stroke
 				(width 0.12)
@@
 		)
 		(fp_line
-			(start -3.5 2.75)
-			(end 3.05 2.75)
+			(start -2.7 0.9)
+			(end -2.7 -0.899999)
 			(stroke
 				(width 0.12)
-				(type solid)
+				(type default)
 			)
 			(layer "F.SilkS")
 		)
 		(fp_line
-			(start -2.7 0.9)
-			(end -2.7 -0.9)
+			(start -3.499999 2.75)
+			(end 3.05 2.749999)
 			(stroke
 				(width 0.12)
-				(type default)
+				(type solid)
 			)
 			(layer "F.SilkS")
 		)
 		(fp_line
-			(start 2.7 0.9)
+			(start 2.7 0.899999)
 			(end 2.7 -0.9)
 			(stroke
@@
 		)
 		(fp_line
-			(start 3.05 2.75)
-			(end 3.5 2.3)
+			(start 3.5 2.3)
+			(end 3.499999 -2.75)
 			(stroke
 				(width 0.12)
@@
 		)
 		(fp_line
-			(start 3.5 2.3)
-			(end 3.5 -2.75)
+			(start 3.05 2.749999)
+			(end 3.5 2.3)
 			(stroke
 				(width 0.12)
@@
 		)
 		(fp_line
-			(start -3.45 -2.75)
-			(end -3.45 2.75)
+			(start -3.45 -2.749999)
+			(end -3.449998 2.75)
 			(stroke
 				(width 0.05)
@@
 		)
 		(fp_line
-			(start -3.45 2.75)
-			(end 3.45 2.75)
+			(start -3.449998 2.75)
+			(end 3.45 2.749999)
 			(stroke
 				(width 0.05)
@@
 		)
 		(fp_line
-			(start 3.45 -2.75)
-			(end -3.45 -2.75)
+			(start 3.449998 -2.75)
+			(end -3.45 -2.749999)
 			(stroke
 				(width 0.05)
@@
 		)
 		(fp_line
-			(start 3.45 2.75)
-			(end 3.45 -2.75)
+			(start 3.45 2.749999)
+			(end 3.449998 -2.75)
 			(stroke
 				(width 0.05)
@@
 		)
 		(fp_line
-			(start -2.5 2.5)
-			(end 2.5 2.5)
+			(start 2.5 -2.5)
+			(end -2.5 -2.5)
 			(stroke
 				(width 0.1)
@@
 		)
 		(fp_line
-			(start 2.5 -2.5)
-			(end -2.5 -2.5)
+			(start -2.5 2.5)
+			(end 2.5 2.5)
 			(stroke
 				(width 0.1)
@@
 		(fp_line
 			(start 2.5 1.5)
-			(end 1.5 2.5)
+			(end 1.499999 2.499999)
 			(stroke
 				(width 0.1)
@@
 		)
 		(fp_text user "1"
-			(at -4 -1.6 0)
+			(at -4 -1.600001 50)
 			(unlocked yes)
 			(layer "F.SilkS")
@@
 		)
 		(fp_text user "${REFERENCE}"
-			(at 0 0 0)
+			(at 0 0 50)
 			(layer "F.Fab")
 			(effects
@@
 		)
 		(pad "1" smd roundrect
-			(at -2.45 -1.65)
+			(at -2.45 -1.65 50)
 			(size 1.5 0.9)
 			(layers "F.Cu" "F.Mask" "F.Paste")
@@
 		)
 		(pad "2" smd roundrect
-			(at -2.45 1.65)
+			(at -2.45 1.650001 50)
 			(size 1.5 0.9)
 			(layers "F.Cu" "F.Mask" "F.Paste")
@@
 		)
 		(pad "3" smd roundrect
-			(at 2.45 1.65)
+			(at 2.45 1.65 50)
 			(size 1.5 0.9)
 			(layers "F.Cu" "F.Mask" "F.Paste")
@@
 		)
 		(pad "4" smd roundrect
-			(at 2.45 -1.65)
+			(at 2.45 -1.650001 50)
 			(size 1.5 0.9)
 			(layers "F.Cu" "F.Mask" "F.Paste")
@@
 	)
 	(segment
+		(start 216.625 43.715)
+		(end 216.625 44.261)
+		(width 0.2)
+		(layer "F.Cu")
+		(net 18)
+	)
+	(segment
 		(start 209.929 50.957)
-		(end 204.671 50.957)
+		(end 202.795265 50.957)
 		(width 0.2)
 		(layer "F.Cu")
@@
 	)
 	(segment
-		(start 216.625 43.715)
-		(end 216.625 44.261)
+		(start 202.795265 50.957)
+		(end 202.240856 50.402591)
 		(width 0.2)
 		(layer "F.Cu")
@@
 	)
 	(segment
-		(start 199.771 65.725)
-		(end 199.681 65.815)
+		(start 199.771 58.125553)
+		(end 199.771 65.725)
 		(width 0.2)
 		(layer "F.Cu")
@@
 	)
 	(segment
-		(start 199.771 54.257)
-		(end 199.771 65.725)
+		(start 201.619144 56.277409)
+		(end 199.771 58.125553)
+		(width 0.2)
+		(layer "F.Cu")
+		(net 19)
+	)
+	(segment
+		(start 199.771 65.725)
+		(end 199.681 65.815)
 		(width 0.2)
 		(layer "F.Cu")
@@
 	)
 	(segment
-		(start 204.597 54.331)
-		(end 204.597 54.383)
+		(start 236.765 83.339)
+		(end 236.855 83.339)
 		(width 0.2)
 		(layer "F.Cu")
@@
 	)
 	(segment
-		(start 236.765 83.339)
-		(end 236.855 83.339)
+		(start 246.417 70.131)
+		(end 246.507 70.131)
 		(width 0.2)
 		(layer "F.Cu")
@@
 	)
 	(segment
-		(start 246.417 70.131)
-		(end 246.507 70.131)
+		(start 204.768803 52.523791)
+		(end 204.597 52.695594)
+		(width 0.2)
+		(layer "F.Cu")
+		(net 112)
+	)
+	(segment
+		(start 206.404209 52.523791)
+		(end 204.768803 52.523791)
 		(width 0.2)
 		(layer "F.Cu")
@@
 	)
 	(segment
-		(start 204.671 54.257)
-		(end 204.597 54.331)
+		(start 206.858 52.07)
+		(end 206.404209 52.523791)
+		(width 0.2)
+		(layer "F.Cu")
+		(net 112)
+	)
+	(segment
+		(start 207.01 52.07)
+		(end 206.858 52.07)
 		(width 0.2)
 		(layer "F.Cu")
@@
 	)
 	(via
-		(at 204.671 54.257)
+		(at 207.01 52.07)
 		(size 0.6)
 		(drill 0.3)

Commit message: .
Parts:
- removed D1, D14, D15, D16, D17, D18, D19, D2: WS2812B, LED_SMD:LED_WS2812B_PLCC4_5.0x5.0mm_P3.2mm
- removed J5: Top Interface, Connector_PinSocket_2.54mm:PinSocket_1x12_P2.54mm_Vertical
- removed J6: Top, Connector_PinHeader_2.54mm:PinHeader_1x12_P2.54mm_Horizontal
- added D13: WS2812B, LED_SMD:LED_WS2812B_PLCC4_5.0x5.0mm_P3.2mm, F.Cu at (-67.8, 108.0)
- added SW1: SW_SPDT, Button_Switch_THT:SW_Slide_SPDT_Angled_CK_OS102011MA1Q, F.Cu at (76.3, 38.8)
- added mouse-bite-2.54mm-slot: VAL**, MouseBites:mouse-bite-2.54mm-slot, F.Cu at (113.7, 121.9)
- added mouse-bite-2.54mm-slot: VAL**, MouseBites:mouse-bite-2.54mm-slot, F.Cu at (113.7, 44.5)
- added mouse-bite-2.54mm-slot: VAL**, MouseBites:mouse-bite-2.54mm-slot, F.Cu at (113.7, 83.2)
- J1, J2: moved to F.Cu
- moved J3 212.2 mm to (-40.0, 87.0)
- moved J13 160.1 mm to (-65.0, 51.8)
- moved J1 157.9 mm to (-49.2, 87.0), turned to 0 degrees
- moved J4 153.9 mm to (-35.4, 87.0)
- moved J12 149.8 mm to (-55.8, 51.8)
- moved J11 141.9 mm to (-69.6, 51.8)
- moved R8 140.1 mm to (-61.4, 109.2), turned to 0 degrees
- moved D12 134.7 mm to (-61.4, 106.2)
- moved J8 132.7 mm to (-23.9, 29.2), turned to 0 degrees
- moved J10 131.6 mm to (-60.4, 51.8)
- moved C8 111.0 mm to (-43.3, 78.7)
- moved C7 110.6 mm to (-43.3, 75.7), turned to 0 degrees
- moved C5 110.5 mm to (-43.3, 69.6), turned to 0 degrees
- moved C3 109.0 mm to (-43.3, 63.6), turned to 0 degrees
- moved C9 107.4 mm to (-36.4, 69.4), turned to 0 degrees
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Connections:
- net /RS485 Interface/232_RX renamed /Front PCB/RS485 Interface/232_RX
- net /RS485 Interface/232_TX renamed /Front PCB/RS485 Interface/232_TX
- net /RS485 Interface/DIR renamed /Front PCB/RS485 Interface/DIR
- net /RS485 Interface/Data_A renamed /Front PCB/RS485 Interface/Data_A
- net /RS485 Interface/Data_B renamed /Front PCB/RS485 Interface/Data_B
- D4 pad 1: +Solar -> Net-(D4-K)
- D5 pad 1: +Solar -> Net-(D4-K)
- D6 pad 1: +Solar -> Net-(D4-K)
- D7 pad 1: +Solar -> Net-(D4-K)
- D8 pad 1: +Solar -> Net-(D4-K)
- D9 pad 1: +Solar -> Net-(D4-K)
- J11 pad 16: /Front PCB/Shrimp/37 -> /Front PCB/NeoPixle_Out
Routing:
- net /Front PCB/Heart Beat: track 37.7 -> 0.00 mm
- net Net-(D4-K): track 0.00 -> 32.4 mm
- net /Top PCB/NeoPixle_In: track 29.0 -> 0.00 mm
- net Net-(D11-K): track 25.7 -> 0.00 mm
- net Net-(D1-DOUT): track 23.3 -> 0.00 mm
- net +5V: track 23.0 -> 0.00 mm, vias 2 -> 0
- net Net-(D18-DIN): track 22.5 -> 0.00 mm
- net Net-(D18-DOUT): track 22.1 -> 0.00 mm
- net Net-(D1-DIN): track 21.6 -> 0.00 mm
- net Net-(D16-DOUT): track 20.6 -> 0.00 mm
- net Net-(D14-DOUT): track 17.9 -> 0.00 mm
- net Net-(U1-VSENSE): track 10.5 -> 0.00 mm
- net Net-(D15-DOUT): track 10.3 -> 0.00 mm
- net +Solar: track 45.8 -> 36.8 mm
- net Net-(U1-COMP): track 5.58 -> 0.00 mm
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- removed copper zone on F.Cu, net Back PCB +5V
- removed copper zone on F.Cu, net Front PCB +5V
- removed copper zone on B.Cu, net Front PCB GND
- removed copper zone on F.Cu, net Top PCB +5V
- removed copper zone on B.Cu, net Top PCB GND
Other:
- board size 191.8 x 100 mm -> 91.4 x 99.1 mm
