File: Main PCB KiCAD/Buoy PCB.kicad_pcb (KiCad board)
At the start: 2 copper layers, 91.4 x 99.1 mm, 49 parts, among them J1 Front B, J10 P2, J11 P4, J12 P3, J13 P5, J2 Front A, J3 Back B, J4 Back A, J7 Solar in, J8 RS485, J9 Bench Power, SW1 SW_SPDT, U1 TPS54331D, U2 MAX3072E

Commit message: .
Parts:
- added D14: WS2812B, LED_SMD:LED_WS2812B_PLCC4_5.0x5.0mm_P3.2mm, F.Cu at (98.4, 36.8)
- added D15: WS2812B, LED_SMD:LED_WS2812B_PLCC4_5.0x5.0mm_P3.2mm, F.Cu at (130.2, 36.8)
- added D16: WS2812B, LED_SMD:LED_WS2812B_PLCC4_5.0x5.0mm_P3.2mm, F.Cu at (152.4, 36.8)
- added NT1: NetTie_2, NetTie:NetTie-2_SMD_Pad0.5mm, B.Cu at (117.5, 121.9)
- added NT2: NetTie_2, NetTie:NetTie-2_SMD_Pad0.5mm, F.Cu at (117.5, 121.9)
- added NT3: NetTie_2, NetTie:NetTie-2_SMD_Pad0.5mm, F.Cu at (117.5, 44.5)
- J1, J2, J3, J4: moved to B.Cu
- mouse-bite-2.54mm-slot (x3): footprint MouseBites:mouse-bite-2.54mm-slot -> KiCad Footprints:MouseBite Slot 2.54 x 2.54mm
- moved J3 205.7 mm to (165.1, 102.9), turned to 180 degrees
- moved D13 169.2 mm to (85.7, 36.8)
- moved D12 168.9 mm to (92.1, 35.6)
- moved R8 168.9 mm to (92.1, 38.7)
- moved J2 159.7 mm to (114.3, 102.9), turned to 180 degrees
- moved J4 157.5 mm to (121.3, 102.9), turned to 180 degrees
- moved J8 137.8 mm to (108.7, 66.7), turned to 90 degrees
- moved J1 120.1 mm to (69.8, 102.9), turned to 180 degrees
- moved C1 73.2 mm to (29.7, 65.7)
- moved C10 73.2 mm to (36.6, 81.3)
- moved C2 73.2 mm to (36.6, 67.6)
- moved C3 73.2 mm to (29.7, 68.7)
- moved C4 73.2 mm to (29.7, 71.7)
- moved C5 73.2 mm to (29.7, 74.7)
- moved C6 73.2 mm to (29.7, 77.7)
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Connections:
- D13 pad 2: unconnected-(D13-DOUT-Pad2) -> Net-(D13-DOUT)
- J1 pad 2: Front PCB GND -> Front PCB +5V
- J1 pad 3: Front PCB +5V -> Front PCB GND
- J2 pad 2: Front PCB GND -> Front PCB +5V
- J2 pad 3: Front PCB +5V -> Front PCB GND
- J2 pad 5: unconnected-(J2-Pin_5-Pad5) -> /Front PCB/NeoPixle_Connect_out
- J3 pad 2: Back PCB GND -> Back PCB +5V
- J3 pad 3: Back PCB +5V -> Back PCB GND
- J4 pad 2: Back PCB GND -> Back PCB +5V
- J4 pad 3: Back PCB +5V -> Back PCB GND
- J4 pad 5: unconnected-(J4-Pin_5-Pad5) -> /Back PCB/NeoPixle_Connect_in
Routing:
- net Back PCB GND: track 0.00 -> 40.2 mm
- net Net-(D15-DOUT): track 0.00 -> 28.5 mm
- net /Front PCB/NeoPixle_Connect_out: track 0.00 -> 23.5 mm
- net Front PCB +5V: track 0.00 -> 21.9 mm
- net Back PCB +5V: track 0.00 -> 21.9 mm
- net /Back PCB/NeoPixle_Connect_in: track 0.00 -> 20.3 mm
- net Net-(D13-DOUT): track 0.00 -> 19.0 mm
- net Front PCB GND: track 0.00 -> 16.8 mm
- net Top PCB GND: track 0.00 -> 13.5 mm
- net Top PCB +5V: track 0.00 -> 13.4 mm
- net Net-(D12-A): track 0.00 -> 5.49 mm, vias 0 -> 2
Other:
- board size 91.4 x 99.1 mm -> 99.1 x 99.1 mm

Commit message: .
Parts:
- removed J10: P2, Connector_PinSocket_2.54mm:PinSocket_1x08_P2.54mm_Vertical
- removed J11: P4, Connector_PinSocket_2.54mm:PinSocket_1x16_P2.54mm_Vertical
- removed J12: P3, Connector_PinSocket_2.54mm:PinSocket_1x08_P2.54mm_Vertical
- removed J13: P5, Connector_PinSocket_2.54mm:PinSocket_1x16_P2.54mm_Vertical
- added U3: Pimoroni PGA2350, KiCad Footprints:PGA2350, F.Cu at (92.7, 87.0)
