File: Main PCB KiCAD/Buoy PCB.kicad_pcb (KiCad board)
At the start: 2 copper layers, 99.1 x 99.1 mm, 52 parts, among them J1 Front B, J2 Front A, J3 Back B, J4 Back A, J7 Solar in, J8 RS485, J9 Bench Power, SW1 SW_SPDT, U1 TPS54331D, U2 MAX3072E, U3 Pimoroni PGA2350

Commit message: .
Parts:
- added D17: 20V 1A, Diode_SMD:D_0805_2012Metric_Pad1.15x1.40mm_HandSolder, F.Cu at (72.4, 76.2)
- added SW2: Reset, Button_Switch_THT:SW_PUSH-12mm, F.Cu at (31.4, 126.7)
- added SW3: Boot, Button_Switch_THT:SW_PUSH-12mm, F.Cu at (31.4, 142.2)
- moved J1 0.64 mm to (70.5, 102.9)
- moved J2 0.63 mm to (113.7, 102.9)
- moved J3 0.63 mm to (164.5, 102.9)
Connections:
- C2 pad 2: GND -> Front PCB GND
- C3 pad 2: GND -> Front PCB GND
- D12 pad 1: GND -> Front PCB GND
- D13 pad 3: Top PCB GND -> Front PCB GND
- D14 pad 3: Top PCB GND -> Front PCB GND
- D3 pad 1: GND -> Front PCB GND
- J7 pad 10: GND -> Front PCB GND
- J7 pad 12: GND -> Front PCB GND
- J7 pad 2: GND -> Front PCB GND
- J7 pad 4: GND -> Front PCB GND
- J7 pad 6: GND -> Front PCB GND
- J7 pad 8: GND -> Front PCB GND
- J9 pad 2: GND -> Front PCB GND
- U3 pad 1: Net-(U3-GND-Pad1) -> Front PCB GND
- U3 pad 10: Net-(U3-GND-Pad1) -> Front PCB GND
- U3 pad 11: unconnected-(U3-GP2-Pad11) -> /Front PCB/UART1_TX
- U3 pad 12: Net-(U3-GND-Pad1) -> Front PCB GND
- U3 pad 13: /Front PCB/Heart Beat -> /Front PCB/UART0_TX
- U3 pad 19: Net-(U3-GND-Pad1) -> Front PCB GND
- U3 pad 2: unconnected-(U3-GP1-Pad2) -> /Front PCB/UART0_RX
- U3 pad 21: unconnected-(U3-GP4-Pad21) -> /Front PCB/UART1_RX
- U3 pad 22: unconnected-(U3-GP3-Pad22) -> /Front PCB/UART1_TX_EN
- U3 pad 3: unconnected-(U3-VBUS-Pad3) -> +5V
- U3 pad 31: /Front PCB/NeoPixle_Out -> unconnected-(U3-GP39-Pad31)
- U3 pad 41: unconnected-(U3-GP14-Pad41) -> /Front PCB/NeoPixle_Out
- U3 pad 5: unconnected-(U3-RUN-Pad5) -> Net-(U3-RUN)
- U3 pad 55: Net-(U3-GND-Pad1) -> Front PCB GND
- U3 pad 6: unconnected-(U3-USB_D+-Pad6) -> Net-(J5-D+)
- U3 pad 64: Net-(U3-GND-Pad1) -> Front PCB GND
- U3 pad 7: unconnected-(U3-USB_D--Pad7) -> Net-(J5-D-)
- U3 pad 8: unconnected-(U3-BOOTSEL-Pad8) -> Net-(U3-BOOTSEL)
Routing:
- net Back PCB GND: track 40.2 -> 24.8 mm
- net Top PCB GND: track 13.5 -> 0.00 mm
- net Front PCB GND: track 16.8 -> 12.0 mm, vias 0 -> 3
- added copper zone on B.Cu, net Back PCB GND
- added copper zone on B.Cu, net Front PCB GND

Commit message: .
Parts:
- removed D10: 1N5819HW-FDICT, Diode_SMD:D_SOD-123
- removed JP2: RS485 - Power, Jumper:SolderJumper-2_P1.3mm_Bridged_RoundedPad1.0x1.5mm
- removed NT1, NT2, NT3: NetTie_2, NetTie:NetTie-2_SMD_Pad0.5mm
- removed SW2: Reset, Button_Switch_THT:SW_PUSH-12mm
- removed SW3: Boot, Button_Switch_THT:SW_PUSH-12mm
- removed U3: Pimoroni PGA2350, KiCad Footprints:PGA2350
- added A1: Adafruit_Feather_M0_RFM9x_LoRa_Radio, Module:Adafruit_Feather_M0_RFM, B.Cu at (82.0, 79.4)
- J7: footprint Connector_JST:JST_PH_S12B-PH-K_1x12_P2.00mm_Horizontal -> Connector_JST:JST_EH_S12B-EH_1x12_P2.50mm_Horizontal; moved to B.Cu
- J8: value RS485 -> Conn_01x09; footprint Connector_JST:JST_PH_S8B-PH-K_1x08_P2.00mm_Horizontal -> Connector_JST:JST_EH_S9B-EH_1x09_P2.50mm_Horizontal; moved to B.Cu
- J9: value Bench Power -> Conn_01x02; footprint Connector_JST:JST_PH_S2B-PH-K_1x02_P2.00mm_Horizontal -> Connector_JST:JST_EH_S2B-EH_1x02_P2.50mm_Horizontal; moved to B.Cu
- JP1: value Terminator -> RS485 - Power; footprint Jumper:SolderJumper-2_P1.3mm_Open_RoundedPad1.0x1.5mm -> Jumper:SolderJumper-2_P1.3mm_Bridged_RoundedPad1.0x1.5mm
- SW1: moved to B.Cu
- moved D3 135.9 mm to (160.7, 35.6), turned to -90 degrees
- moved C3 132.1 mm to (153.7, 114.3)
- moved C1 131.2 mm to (155.6, 102.9)
- moved C2 124.5 mm to (153.7, 109.9)
- moved C8 121.3 mm to (146.7, 51.4), turned to 180 degrees
- moved R1 120.1 mm to (160.7, 39.4), turned to 90 degrees
- moved R3 117.1 mm to (155.6, 105.4)
- moved J7 116.5 mm to (159.4, 129.5), turned to 90 degrees
- moved R2 114.4 mm to (151.8, 105.4)
- moved C9 113.5 mm to (146.7, 47.0)
- moved D4 108.8 mm to (153.7, 129.5), turned to 0 degrees
- moved C10 107.5 mm to (138.4, 47.0)
- moved D5 104.2 mm to (153.7, 127.0), turned to 0 degrees
- moved D6 99.7 mm to (153.7, 124.5), turned to 0 degrees
- moved C4 98.4 mm to (127.9, 78.5)
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Connections:
- net /Front PCB/V_Solar_An renamed /Back PCB/V_Solar_An
- C10 pad 1: +5V -> Net-(SW1-B)
- C2 pad 2: Front PCB GND -> GND
- C3 pad 2: Front PCB GND -> GND
- C8 pad 2: +5V -> Net-(SW1-B)
- C9 pad 1: +5V -> Net-(SW1-B)
- D12 pad 1: Front PCB GND -> GND
- D13 pad 1: Top PCB +5V -> +5V
- D13 pad 3: Front PCB GND -> GND
- D14 pad 1: Top PCB +5V -> +5V
- D14 pad 2: /Front PCB/NeoPixle_Connect_out -> /Back PCB/NeoPixle_Connect_in
- D14 pad 3: Front PCB GND -> GND
- D15 pad 1: Back PCB +5V -> +5V
- D15 pad 3: Back PCB GND -> GND
- D16 pad 1: Back PCB +5V -> +5V
- D16 pad 3: Back PCB GND -> GND
- D3 pad 1: Front PCB GND -> GND
- D4 pad 1: Net-(D4-K) -> +Solar
- D5 pad 1: Net-(D4-K) -> +Solar
- D6 pad 1: Net-(D4-K) -> +Solar
- D7 pad 1: Net-(D4-K) -> +Solar
- D8 pad 1: Net-(D4-K) -> +Solar
- D9 pad 1: Net-(D4-K) -> +Solar
- J1 pad 1: Front PCB +5V -> +5V
- J1 pad 2: Front PCB +5V -> +5V
- J1 pad 3: Front PCB GND -> GND
- J1 pad 4: Front PCB GND -> GND
- J2 pad 1: Front PCB +5V -> +5V
- J2 pad 10: unconnected-(J2-Pin_10-Pad10) -> Net-(J2-Pin_10)
- J2 pad 11: unconnected-(J2-Pin_11-Pad11) -> Net-(J2-Pin_11)
- J2 pad 12: unconnected-(J2-Pin_12-Pad12) -> Net-(J2-Pin_12)
- J2 pad 2: Front PCB +5V -> +5V
- J2 pad 3: Front PCB GND -> GND
- J2 pad 4: Front PCB GND -> GND
- J2 pad 5: /Front PCB/NeoPixle_Connect_out -> /Back PCB/NeoPixle_Connect_in
- J2 pad 6: unconnected-(J2-Pin_6-Pad6) -> Net-(J2-Pin_6)
- J2 pad 7: unconnected-(J2-Pin_7-Pad7) -> Net-(J2-Pin_7)
- J2 pad 8: unconnected-(J2-Pin_8-Pad8) -> Net-(J2-Pin_8)
- J2 pad 9: unconnected-(J2-Pin_9-Pad9) -> Net-(J2-Pin_9)
- J3 pad 1: Back PCB +5V -> +5V
- J3 pad 2: Back PCB +5V -> +5V
- J3 pad 3: Back PCB GND -> GND
- J3 pad 4: Back PCB GND -> GND
- J4 pad 1: Back PCB +5V -> +5V
- J4 pad 10: unconnected-(J4-Pin_10-Pad10) -> Net-(J2-Pin_10)
- J4 pad 11: unconnected-(J4-Pin_11-Pad11) -> Net-(J2-Pin_11)
- J4 pad 12: unconnected-(J4-Pin_12-Pad12) -> Net-(J2-Pin_12)
- J4 pad 2: Back PCB +5V -> +5V
- J4 pad 3: Back PCB GND -> GND
- J4 pad 4: Back PCB GND -> GND
- J4 pad 6: unconnected-(J4-Pin_6-Pad6) -> Net-(J2-Pin_6)
- J4 pad 7: unconnected-(J4-Pin_7-Pad7) -> Net-(J2-Pin_7)
- J4 pad 8: unconnected-(J4-Pin_8-Pad8) -> Net-(J2-Pin_8)
- J4 pad 9: unconnected-(J4-Pin_9-Pad9) -> Net-(J2-Pin_9)
- J7 pad 10: Front PCB GND -> GND
- J7 pad 12: Front PCB GND -> GND
- J7 pad 2: Front PCB GND -> GND
- J7 pad 4: Front PCB GND -> GND
- J7 pad 6: Front PCB GND -> GND
- J7 pad 8: Front PCB GND -> GND
- J8 pad 8: GND -> Net-(J8-Pin_8)
- J9 pad 1: Net-(D10-A) -> Net-(D17-A)
- J9 pad 2: Front PCB GND -> GND
- JP1 pad 1: /Front PCB/RS485 Interface/Data_B -> Net-(J8-Pin_1)
- JP1 pad 2: Net-(JP1-B) -> +5V
- L1 pad 2: +5V -> Net-(SW1-B)
- R5 pad 1: +5V -> Net-(SW1-B)
- R7 pad 1: /Front PCB/RS485 Interface/Data_A -> /Front PCB/RS485 Interface/Data_B
- R7 pad 2: Net-(JP1-B) -> Net-(J8-Pin_8)
- SW1 pad 1: +Solar -> +5V
- SW1 pad 2: Net-(D4-K) -> Net-(SW1-B)
Routing:
- net +Solar: track 36.8 -> 95.8 mm
- net Net-(J2-Pin_9): track 0.00 -> 57.1 mm
- net Net-(J2-Pin_10): track 0.00 -> 53.0 mm
- net Net-(J2-Pin_11): track 0.00 -> 47.1 mm
- net Net-(J2-Pin_12): track 0.00 -> 43.0 mm
- net GND: track 0.00 -> 35.3 mm, vias 0 -> 12
- net +5V: track 0.00 -> 32.5 mm, vias 0 -> 4
- net Net-(D4-K): track 32.4 -> 0.00 mm
- net /Front PCB/Heart Beat: track 0.00 -> 32.4 mm
- net /Back PCB/NeoPixle_Connect_in: track 20.3 -> 48.5 mm, vias 0 -> 2
- net /Front PCB/NeoPixle_Out: track 0.00 -> 25.3 mm
- net Back PCB GND: track 24.8 -> 0.00 mm
- net Net-(J2-Pin_8): track 0.00 -> 24.8 mm
- net /Front PCB/NeoPixle_Connect_out: track 23.5 -> 0.00 mm
- net /Front PCB/RS485 Interface/Data_B: track 0.00 -> 23.0 mm
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- added copper zone on F.Cu, net +5V
- added copper zone on B.Cu, net GND
- removed copper zone on B.Cu, net Back PCB GND
- removed copper zone on B.Cu, net Front PCB GND

Commit message: .
Parts:
- removed C10: 47μF, Capacitor_SMD:CP_Elec_5x5.9
- removed C4: 10nF, Capacitor_SMD:C_0805_2012Metric_Pad1.18x1.45mm_HandSolder
- removed C5: 10pF, Capacitor_SMD:C_0805_2012Metric_Pad1.18x1.45mm_HandSolder
- removed C6: 1nF, Capacitor_SMD:C_0805_2012Metric_Pad1.18x1.45mm_HandSolder
- removed C7: 0.1uF, Capacitor_SMD:C_0805_2012Metric_Pad1.18x1.45mm_HandSolder
- removed D11: SS34, Diode_SMD:D_SMA_Handsoldering
- removed L1: 8.2uH, Inductor_SMD:L_Taiyo-Yuden_NR-60xx_HandSoldering
- removed R4: 29.4k, Resistor_SMD:R_0805_2012Metric_Pad1.20x1.40mm_HandSolder
- removed R5: 10k2, Resistor_SMD:R_0805_2012Metric_Pad1.20x1.40mm_HandSolder
- removed R6: 1k96, Resistor_SMD:R_0805_2012Metric_Pad1.20x1.40mm_HandSolder
- removed U1: TPS54331D, Package_SO:TI_SO-PowerPAD-8_ThermalVias
- added BT1: Battery_Cell, Battery:BatteryHolder_Keystone_1042_1x18650, F.Cu at (154.2, 88.4)
- added BT2: Battery_Cell, Battery:BatteryHolder_Keystone_1042_1x18650, F.Cu at (131.5, 88.4)
- added JP2: Termination, Jumper:SolderJumper-2_P1.3mm_Bridged_RoundedPad1.0x1.5mm, F.Cu at (80.6, 127.6)
- added R9: Poka Yoke UART, KiCad Footprints:Poka yoke UART Solder, F.Cu at (88.9, 123.0)
- C8, C9: moved to B.Cu
- J8: value Conn_01x09 -> RS485; footprint Connector_JST:JST_EH_S9B-EH_1x09_P2.50mm_Horizontal -> Connector_JST:JST_EH_S8B-EH_1x08_P2.50mm_Horizontal
- J9: value Conn_01x02 -> BenchTop Power
- JP1: value RS485 - Power -> RS485 Power
- moved C9 9.09 mm to (154.9, 43.2), turned to 180 degrees
- moved C8 8.84 mm to (154.9, 48.3), turned to 0 degrees
- moved J8 2.50 mm to (75.6, 112.0)
- moved R7 2.01 mm to (84.5, 127.6)
- moved JP1 1.91 mm to (80.6, 118.7)
Connections:
- A1 pad 14: unconnected-(A1-RX/D0-Pad14) -> /Back PCB/UART0_RX
- A1 pad 15: unconnected-(A1-TX/D1-Pad15) -> /Back PCB/UART0_TX
- A1 pad 22: unconnected-(A1-D10-Pad22) -> /Front PCB/UART1_TX_EN
- A1 pad 23: unconnected-(A1-D11-Pad23) -> /Front PCB/UART1_RX
- A1 pad 24: unconnected-(A1-D12-Pad24) -> /Front PCB/UART1_TX
- A1 pad 28: unconnected-(A1-VBAT-Pad28) -> +Bat
- A1 pad 5: /Front PCB/V_Solar_An -> /Back PCB/V_Solar_An
- C8 pad 2: Net-(SW1-B) -> +5V
- C9 pad 1: Net-(SW1-B) -> +5V
- J2 pad 10: Net-(J2-Pin_10) -> /Back PCB/Data_B
- J2 pad 6: Net-(J2-Pin_6) -> /Back PCB/V_Solar_An
- J2 pad 7: Net-(J2-Pin_7) -> /Back PCB/UART0_RX
- J2 pad 8: Net-(J2-Pin_8) -> /Back PCB/UART0_TX
- J2 pad 9: Net-(J2-Pin_9) -> /Back PCB/Data_A
- J4 pad 10: Net-(J2-Pin_10) -> /Back PCB/Data_B
- J4 pad 6: Net-(J2-Pin_6) -> /Back PCB/V_Solar_An
- J4 pad 7: Net-(J2-Pin_7) -> /Back PCB/UART0_RX
- J4 pad 8: Net-(J2-Pin_8) -> /Back PCB/UART0_TX
- J4 pad 9: Net-(J2-Pin_9) -> /Back PCB/Data_A
- J8 pad 2: /Front PCB/RS485 Interface/Data_A -> /Back PCB/Data_A
- J8 pad 3: /Front PCB/RS485 Interface/Data_B -> /Back PCB/Data_B
- J8 pad 6: /Front PCB/RS485 Interface/Data_A -> /Back PCB/Data_A
- J8 pad 7: /Front PCB/RS485 Interface/Data_B -> /Back PCB/Data_B
- J8 pad 8: Net-(J8-Pin_8) -> GND
- R7 pad 1: /Front PCB/RS485 Interface/Data_B -> /Back PCB/Data_A
- R7 pad 2: Net-(J8-Pin_8) -> Net-(JP2-B)
- SW1 pad 2: Net-(SW1-B) -> unconnected-(SW1-B-Pad2)
- U2 pad 1: /Front PCB/RS485 Interface/232_RX -> Net-(U2-RO)
- U2 pad 2: /Front PCB/RS485 Interface/DIR -> /Front PCB/UART1_TX_EN
- U2 pad 3: /Front PCB/RS485 Interface/DIR -> /Front PCB/UART1_TX_EN
- U2 pad 4: /Front PCB/RS485 Interface/232_TX -> Net-(U2-DI)
- U2 pad 6: /Front PCB/RS485 Interface/Data_A -> /Back PCB/Data_A
- U2 pad 7: /Front PCB/RS485 Interface/Data_B -> /Back PCB/Data_B
Routing:
- net /Back PCB/Data_A: track 0.00 -> 163.3 mm, vias 0 -> 1
- net /Back PCB/V_Solar_An: track 4.37 -> 160.1 mm, vias 0 -> 1
- net /Back PCB/Data_B: track 0.00 -> 155.5 mm
- net /Front PCB/UART1_TX_EN: track 0.00 -> 81.6 mm, vias 0 -> 1
- net /Front PCB/UART1_RX: track 0.00 -> 79.3 mm, vias 0 -> 1
- net /Front PCB/UART1_TX: track 0.00 -> 74.3 mm, vias 0 -> 1
- net /Back PCB/UART0_TX: track 0.00 -> 64.3 mm
- net Net-(J2-Pin_9): track 57.1 -> 0.00 mm
- net /Back PCB/UART0_RX: track 0.00 -> 55.1 mm
- net Net-(J2-Pin_10): track 53.0 -> 0.00 mm
- net +Bat: track 0.00 -> 29.3 mm
- net GND: track 35.3 -> 63.2 mm, vias 12 -> 10
- net Net-(J2-Pin_8): track 24.8 -> 0.00 mm
- net /Front PCB/RS485 Interface/Data_B: track 23.0 -> 0.00 mm
- net Net-(SW1-B): track 22.2 -> 0.00 mm
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
Commit message: .
Parts:
- added J10: RS485 Addr 0, Connector_JST:JST_EH_S7B-EH_1x07_P2.50mm_Horizontal, B.Cu at (126.0, 114.5)
- added J11: RS485 Addr 1, Connector_JST:JST_EH_S7B-EH_1x07_P2.50mm_Horizontal, B.Cu at (126.0, 90.0)
- added J12: RS485 Addr 2, Connector_JST:JST_EH_S7B-EH_1x07_P2.50mm_Horizontal, B.Cu at (159.5, 93.0)
