File: Main PCB KiCAD/Buoy PCB.kicad_sch (KiCad schematic)
At the start: 5 parts, among them J1 Conn_01x12_Socket, J2 Conn_01x12_Socket, J3 Conn_01x12_Pin, J4 Conn_01x12_Pin

Commit message: Changed Micro
Parts:
- removed XA1: Arduino_Mega2560_Shield, Arduino:Arduino_Mega2560_Shield, symbol Arduino:Arduino_Mega2560_Shield
Other:
- added sheet Arduino Mega (Arduino Mega.kicad_sch)
Changed lines of the file:
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@@
-	)
-	(symbol
-		(lib_id "Arduino:Arduino_Mega2560_Shield")
-		(at 349.25 0 0)
-		(unit 1)
-		(exclude_from_sim no)
-		(in_bom yes)
-		(on_board yes)
-		(dnp no)
-		(fields_autoplaced yes)
-		(property "Reference" "XA1"
-			(at 349.25 60.96 0)
-			(effects
-				(font
-					(size 1.524 1.524)
-				)
-			)
-		)
-		(property "Value" "Arduino_Mega2560_Shield"
-			(at 349.25 63.5 0)
-			(effects
-				(font
-					(size 1.524 1.524)
-				)
-			)
-		)
-		(property "Footprint" "Arduino:Arduino_Mega2560_Shield"
-			(at 367.03 -69.85 0)
-			(effects
-				(font
-					(size 1.524 1.524)
-				)
-				(hide yes)
-			)
-		)
-		(property "Datasheet" ""
-			(at 367.03 -69.85 0)
-			(effects
-				(font
-					(size 1.524 1.524)
-				)
-				(hide yes)
-			)
-		)
-		(property "Description" ""
-			(at 349.25 0 0)
-			(effects
-				(font
-					(size 1.27 1.27)
-				)
-				(hide yes)
-			)
-		)
-		(pin "D19"
-		)
-		(pin "D1"
-		)
-		(pin "D18"
-		)
-		(pin "D17"
-		)
-		(pin "D16"
-		)
-		(pin "D15"
-		)
-		(pin "D14"
-		)
-		(pin "D20"
-		)
-		(pin "D21"
-		)
-		(pin "SDA"
-		)
-		(pin "SCL"
-		)
-		(pin "A0"
-		)
-		(pin "A1"
-		)
-		(pin "A2"
-		)
-		(pin "A3"
-		)
-		(pin "A4"
-		)
-		(pin "A5"
-		)
-		(pin "A6"
-		)
-		(pin "A7"
-		)
-		(pin "A8"
-		)
-		(pin "A9"
-		)
-		(pin "A10"
-		)
-		(pin "A11"
-		)
-		(pin "A12"
-		)
-		(pin "A13"
-		)
-		(pin "A14"
-		)
-		(pin "A15"
-		)
-		(pin "AREF"
-		)
-		(pin "RST1"
-		)
-		(pin "IORF"
-		)
-		(pin "GND1"
-		)
-		(pin "GND2"
-		)
-		(pin "GND3"
-		)
-		(pin "GND5"
-		)
-		(pin "GND6"
-		)
-		(pin "3V3"
-		)
-		(pin "5V1"
-		)
-		(pin "5V3"
-		)
-		(pin "5V4"
-		)
-		(pin "VIN"
-		)
-		(pin "MISO"
-		)
-		(pin "MOSI"
-		)
-		(pin "SCK"
-		)
-		(pin "5V2"
-		)
-		(pin "GND4"
-		)
-		(pin "RST2"
-		)
-		(pin "D2"
-		)
-		(pin "D3"
-		)
-		(pin "D4"
-		)
-		(pin "D5"
-		)
-		(pin "D6"
-		)
-		(pin "D7"
-		)
-		(pin "D8"
-		)
-		(pin "D9"
-		)
-		(pin "D10"
-		)
-		(pin "D11"
-		)
-		(pin "D12"
-		)
-		(pin "D13"
-		)
-		(pin "D22"
-		)
-		(pin "D23"
-		)
-		(pin "D24"
-		)
-		(pin "D25"
-		)
-		(pin "D26"
-		)
-		(pin "D27"
-		)
-		(pin "D28"
-		)
-		(pin "D29"
-		)
-		(pin "D30"
-		)
-		(pin "D31"
-		)
-		(pin "D32"
-		)
-		(pin "D33"
-		)
-		(pin "D34"
-		)
-		(pin "D35"
-		)
-		(pin "D36"
-		)
-		(pin "D37"
-		)
-		(pin "D38"
-		)
-		(pin "D39"
-		)
-		(pin "D40"
-		)
-		(pin "D41"
-		)
-		(pin "D42"
-		)
-		(pin "D43"
-		)
-		(pin "D44"
-		)
-		(pin "D45"
-		)
-		(pin "D46"
-		)
-		(pin "D47"
-		)
-		(pin "D48"
-		)
-		(pin "D49"
-		)
-		(pin "D50"
-		)
-		(pin "D51"
-		)
-		(pin "D52"
-		)
-		(pin "D53"
-		)
-		(pin "D0"
-		)
-		(instances
-			(project ""
-				(path "/a041e2a6-7d41-458c-91f3-753821d3dfe9"
-					(reference "XA1")
-					(unit 1)
-				)
-			)
-		)
 	)
 	(symbol
@@
 				)
 			)
+		)
+	)
+	(sheet
+		(at 384.81 92.71)
+		(size 46.99 34.29)
+		(exclude_from_sim no)
+		(in_bom yes)
+		(on_board yes)
+		(dnp no)
+		(fields_autoplaced yes)
+		(stroke
+			(width 0.1524)
+			(type solid)
+		)
+		(fill
+			(color 0 0 0 0.0000)
+		)
+		(property "Sheetname" "Arduino Mega"
+			(at 384.81 91.9984 0)
+			(effects
+				(font
+					(size 1.27 1.27)
+				)
+				(justify left bottom)
+			)
+		)
+		(property "Sheetfile" "Arduino Mega.kicad_sch"
+			(at 384.81 127.5846 0)
+			(effects
+				(font
+					(size 1.27 1.27)
+				)
+				(justify left top)
+				(hide yes)
+			)
+		)
+		(instances
+			(project "Buoy PCB"
+				(path "/a041e2a6-7d41-458c-91f3-753821d3dfe9"
+					(page "6")
+				)
+			)

Commit message: cleanup
Parts:
- J1: value Conn_01x12_Socket -> Top B
- J2: value Conn_01x12_Socket -> Top A
- J3: value Conn_01x12_Pin -> Bottom B
- J4: value Conn_01x12_Pin -> Bottom A
Connections:
- net +3.3V: no longer J1.1 (Pin_1)
- net +Solar: no longer J1.2 (Pin_2)
- net GND: no longer J1.3 (Pin_3), J1.4 (Pin_4), J1.7 (Pin_7), J2.12 (Pin_12)
- net V_Batt_An: no longer J3.5 (Pin_5)
- net V_Solar_An: no longer J3.6 (Pin_6)
- net +3.3V_bat: no longer names the net of J3.1 (Pin_1)
- net +Solar_Batt: no longer names the net of J3.2 (Pin_2)
- removed net GND_Batt: J3.3 (Pin_3), J3.4 (Pin_4), J3.7 (Pin_7), J4.12 (Pin_12)
Other:
- sheet Arduino Mega ports: added NeoPixle_Out, V_Batt_An, V_Solar_An; removed none
- sheet Top PCB ports: added NeoPixle_In; removed none
- moved on the sheet: J1, J2, J3, J4

Commit message: update
Parts:
- added J5: Top Interface, Connector_PinSocket_2.54mm:PinSocket_1x12_P2.54mm_Vertical, symbol Connector:Conn_01x12_Socket
- added J6: Top, Connector_PinHeader_2.54mm:PinHeader_1x12_P2.54mm_Horizontal, symbol Connector:Conn_01x12_Pin
- J1: value Top B -> Front B
- J2: value Top A -> Front A
- J3: value Bottom B -> Back B
- J4: value Bottom A -> Back A
Connections:
- new net Top PCB/NeoPixle_In: J5.12 (Pin_12)
- new net Top PCB/Top_PCB_+5V: J5.10 (Pin_10)
- new net Top PCB/Top_PCB_GND: J5.11 (Pin_11), J5.9 (Pin_9)
Other:
- added sheet Back PCB (Back PCB.kicad_sch)
- added sheet Front PCB (Front PCB.kicad_sch)
- sheet Top PCB ports: added Top_PCB_+5V, Top_PCB_GND; removed none
- moved on the sheet: J1, J2, J3, J4

Commit message: updates
Other:
- sheet Arduino Mega renamed Shrimp
- sheet Shrimp: file Arduino Mega.kicad_sch -> Shrimp.kicad_sch
- sheet Shrimp ports: added RST_SW, USER_SW GPIO_0; removed none
Changed lines of the file:
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@@
 			(color 0 0 0 0.0000)
 		)
-		(property "Sheetname" "Arduino Mega"
+		(property "Sheetname" "Shrimp"
 			(at 384.81 91.9984 0)
 			(effects
@@
 			)
 		)
-		(property "Sheetfile" "Arduino Mega.kicad_sch"
+		(property "Sheetfile" "Shrimp.kicad_sch"
 			(at 384.81 127.5846 0)
 			(effects
@@
 			)
 		)
+		(pin "RST_SW" input
+			(at 431.8 102.87 0)
+			(effects
+				(font
+					(size 1.27 1.27)
+				)
+				(justify right)
+			)
+		)
+		(pin "USER_SW GPIO_0" input
+			(at 384.81 104.14 180)
+			(effects
+				(font
+					(size 1.27 1.27)
+				)
+				(justify left)
+			)
+		)

Commit message: changes adn updates
Connections:
- net Front PCB/Front_PCB_+5V: now reaches J6.10 (Pin_10)
- net Front PCB/Front_PCB_+5V: now also J1.1 (Pin_1), J1.3 (Pin_3), J2.1 (Pin_1), J2.3 (Pin_3)
- net Front PCB/Front_PCB_GND: now reaches J6.11 (Pin_11)
- net Front PCB/Front_PCB_GND: now also J1.2 (Pin_2), J1.4 (Pin_4), J2.2 (Pin_2), J2.4 (Pin_4), J6.9 (Pin_9)
- net Front PCB/NeoPixle_Out: now reaches J6.12 (Pin_12)
- net Back PCB/Back_PCB_+5V: now reaches J4.1 (Pin_1)
- net Back PCB/Back_PCB_+5V: now also J3.1 (Pin_1), J3.3 (Pin_3), J4.3 (Pin_3)
- net Back PCB/Back_PCB_GND: now reaches J4.2 (Pin_2)
- net Back PCB/Back_PCB_GND: now also J3.2 (Pin_2), J3.4 (Pin_4), J4.4 (Pin_4)
Other:
- removed sheet Battery Charger
- removed sheet RS485 Interface
- removed sheet Shrimp
- removed sheet Solar
- sheet Back PCB ports: added Back_PCB_+5V, Back_PCB_GND; removed none
- sheet Front PCB ports: added Front_PCB_+5V, Front_PCB_GND, NeoPixle_Out; removed none
- moved on the sheet: J1, J2, J3, J4, J5, J6

Commit message: .
Parts:
- removed J5: Top Interface, Connector_PinSocket_2.54mm:PinSocket_1x12_P2.54mm_Vertical, symbol Connector:Conn_01x12_Socket
- removed J6: Top, Connector_PinHeader_2.54mm:PinHeader_1x12_P2.54mm_Horizontal, symbol Connector:Conn_01x12_Pin
Other:
- removed sheet Top PCB
- sheet Front PCB ports: added none; removed NeoPixle_Out

Commit message: .
Parts:
- added NT1, NT2, NT3: NetTie_2, NetTie:NetTie-2_SMD_Pad0.5mm, symbol Device:NetTie_2
Connections:
- net Back PCB/Back_PCB_+5V: now also J3.2 (Pin_2), J4.2 (Pin_2), NT2.2; no longer J3.3 (Pin_3), J4.3 (Pin_3)
- net Back PCB/Back_PCB_GND: now also J3.3 (Pin_3), J4.3 (Pin_3), NT1.2; no longer J3.2 (Pin_2), J4.2 (Pin_2)
- net Front PCB/Front_PCB_+5V: now also J1.2 (Pin_2), J2.2 (Pin_2), NT2.1; no longer J1.3 (Pin_3), J2.3 (Pin_3)
- net Front PCB/Front_PCB_GND: now also J1.3 (Pin_3), J2.3 (Pin_3), NT1.1; no longer J1.2 (Pin_2), J2.2 (Pin_2)
- net Back PCB/NeoPixle_Connect_in: now reaches J4.5 (Pin_5)
- net Back PCB/NeoPixle_Connect_in: now also NT3.2
- net Front PCB/NeoPixle_Connect_out: now reaches J2.5 (Pin_5)
- net Front PCB/NeoPixle_Connect_out: now also NT3.1
Other:
- sheet Back PCB ports: added NeoPixle_Connect_in; removed none
- sheet Front PCB ports: added NeoPixle_Connect_out; removed none
- moved on the sheet: J1, J2, J3, J4

Commit message: .
Parts:
- removed NT1, NT2, NT3: NetTie_2, NetTie:NetTie-2_SMD_Pad0.5mm, symbol Device:NetTie_2
Connections:
- net Front PCB/Front_PCB_+5V is gone; now on net +5V: J1.1 (Pin_1), J1.2 (Pin_2), J2.1 (Pin_1), J2.2 (Pin_2)
- net Front PCB/Front_PCB_GND is gone; now on net GND: J1.3 (Pin_3), J1.4 (Pin_4), J2.3 (Pin_3), J2.4 (Pin_4)
- net Front PCB/NeoPixle_Connect_out is gone; now on net Back PCB/NeoPixle_Connect_in: J2.5 (Pin_5)
- net at J4.10 (Pin_10): now also J2.10 (Pin_10)
- net at J4.11 (Pin_11): now also J2.11 (Pin_11)
- net at J4.12 (Pin_12): now also J2.12 (Pin_12)
- net at J4.6 (Pin_6): now also J2.6 (Pin_6)
- net at J4.7 (Pin_7): now also J2.7 (Pin_7)
- net at J4.8 (Pin_8): now also J2.8 (Pin_8)
- net at J4.9 (Pin_9): now also J2.9 (Pin_9)
- net Back PCB/Back_PCB_+5V renamed +5V
- net Back PCB/Back_PCB_GND renamed GND
Other:
- sheet Back PCB ports: added none; removed Back_PCB_+5V, Back_PCB_GND
- sheet Front PCB ports: added none; removed Front_PCB_+5V, Front_PCB_GND
