File: Main PCB KiCAD/Buoy PCB.kicad_sch (KiCad schematic)
At the start: 4 parts, among them J1 Front B, J2 Front A, J3 Back B, J4 Back A

Commit message: .
Connections:
- net Back PCB/Data_B: now reaches J2.10 (Pin_10), J4.10 (Pin_10)
- net Back PCB/V_Solar_An: now reaches J2.6 (Pin_6), J4.6 (Pin_6)
- net Back PCB/UART0_RX: now reaches J2.7 (Pin_7), J4.7 (Pin_7)
- net Back PCB/UART0_TX: now reaches J2.8 (Pin_8), J4.8 (Pin_8)
- net Back PCB/Data_A: now reaches J2.9 (Pin_9), J4.9 (Pin_9)
Other:
- sheet Back PCB ports: added Data_A, Data_B, UART0_RX, UART0_TX, V_Solar_An; removed none
- sheet Front PCB ports: added Data_A, Data_B, UART0_RX, UART0_TX, V_Solar_An; removed none
Changed lines of the file:
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@@
 	(paper "A4")
 	(junction
+		(at 124.46 113.03)
+		(diameter 0)
+		(color 0 0 0 0)
+	)
+	(junction
 		(at 134.62 134.62)
 		(diameter 0)
@@
 	)
 	(junction
+		(at 109.22 115.57)
+		(diameter 0)
+		(color 0 0 0 0)
+	)
+	(junction
+		(at 124.46 110.49)
+		(diameter 0)
+		(color 0 0 0 0)
+	)
+	(junction
 		(at 134.62 95.25)
 		(diameter 0)
@@
 	)
 	(junction
+		(at 109.22 110.49)
+		(diameter 0)
+		(color 0 0 0 0)
+	)
+	(junction
+		(at 109.22 105.41)
+		(diameter 0)
+		(color 0 0 0 0)
+	)
+	(junction
 		(at 101.6 100.33)
 		(diameter 0)
@@
 	)
 	(junction
+		(at 109.22 107.95)
+		(diameter 0)
+		(color 0 0 0 0)
+	)
+	(junction
 		(at 104.14 92.71)
 		(diameter 0)
@@
 	)
 	(junction
+		(at 124.46 107.95)
+		(diameter 0)
+		(color 0 0 0 0)
+	)
+	(junction
 		(at 132.08 142.24)
 		(diameter 0)
@@
 	)
 	(junction
+		(at 109.22 113.03)
+		(diameter 0)
+		(color 0 0 0 0)
+	)
+	(junction
+		(at 124.46 115.57)
+		(diameter 0)
+		(color 0 0 0 0)
+	)
+	(junction
 		(at 101.6 139.7)
 		(diameter 0)
@@
 		(color 0 0 0 0)
 	)
+	(junction
+		(at 124.46 105.41)
+		(diameter 0)
+		(color 0 0 0 0)
+	)
+	(wire
+		(pts
+			(xy 109.22 115.57) (xy 124.46 115.57)
+		)
+		(stroke
+			(width 0)
+			(type default)
+		)
+	)
 	(wire
 		(pts
@@
 	(wire
 		(pts
+			(xy 93.98 107.95) (xy 109.22 107.95)
+		)
+		(stroke
+			(width 0)
+			(type default)
+		)
+	)
+	(wire
+		(pts
 			(xy 109.22 102.87) (xy 124.46 102.87)
 		)
@@
 	(wire
 		(pts
+			(xy 124.46 105.41) (xy 142.24 105.41)
+		)
+		(stroke
+			(width 0)
+			(type default)
+		)
+	)
+	(wire
+		(pts
 			(xy 132.08 100.33) (xy 132.08 139.7)
 		)
@@
 	(wire
 		(pts
-			(xy 109.22 115.57) (xy 124.46 115.57)
-		)
-		(stroke
-			(width 0)
-			(type default)
-		)
-	)
-	(wire
-		(pts
 			(xy 109.22 113.03) (xy 124.46 113.03)
 		)
@@
 	(wire
 		(pts
+			(xy 93.98 105.41) (xy 109.22 105.41)
+		)
+		(stroke
+			(width 0)
+			(type default)
+		)
+	)
+	(wire
+		(pts
 			(xy 104.14 95.25) (xy 109.22 95.25)
 		)
@@
 	(wire
 		(pts
+			(xy 93.98 113.03) (xy 109.22 113.03)
+		)
+		(stroke
+			(width 0)
+			(type default)
+		)
+	)
+	(wire
+		(pts
+			(xy 93.98 110.49) (xy 109.22 110.49)
+		)
+		(stroke
+			(width 0)
+			(type default)
+		)
+	)
+	(wire
+		(pts
 			(xy 132.08 142.24) (xy 132.08 175.26)
 		)
@@
 	(wire
 		(pts
+			(xy 124.46 113.03) (xy 142.24 113.03)
+		)
+		(stroke
+			(width 0)
+			(type default)
+		)
+	)
+	(wire
+		(pts
 			(xy 104.14 137.16) (xy 104.14 134.62)
 		)
@@
 	(wire
 		(pts
+			(xy 93.98 115.57) (xy 109.22 115.57)
+		)
+		(stroke
+			(width 0)
+			(type default)
+		)
+	)
+	(wire
+		(pts
 			(xy 104.14 134.62) (xy 109.22 134.62)
 		)
@@
 	(wire
 		(pts
+			(xy 124.46 110.49) (xy 142.24 110.49)
+		)
+		(stroke
+			(width 0)
+			(type default)
+		)
+	)
+	(wire
+		(pts
 			(xy 109.22 137.16) (xy 104.14 137.16)
 		)
@@
 	(wire
 		(pts
+			(xy 124.46 115.57) (xy 142.24 115.57)
+		)
+		(stroke
+			(width 0)
+			(type default)
+		)
+	)
+	(wire
+		(pts
 			(xy 124.46 102.87) (xy 142.24 102.87)
+		)
+		(stroke
+			(width 0)
+			(type default)
+		)
+	)
+	(wire
+		(pts
+			(xy 124.46 107.95) (xy 142.24 107.95)
 		)
 		(stroke
@@
 			)
 		)
+		(pin "V_Solar_An" output
+			(at 142.24 105.41 180)
+			(effects
+				(font
+					(size 1.27 1.27)
+				)
+				(justify left)
+			)
+		)
+		(pin "UART0_RX" bidirectional
+			(at 142.24 107.95 180)
+			(effects
+				(font
+					(size 1.27 1.27)
+				)
+				(justify left)
+			)
+		)
+		(pin "UART0_TX" bidirectional
+			(at 142.24 110.49 180)
+			(effects
+				(font
+					(size 1.27 1.27)
+				)
+				(justify left)
+			)
+		)
+		(pin "Data_A" bidirectional
+			(at 142.24 113.03 180)
+			(effects
+				(font
+					(size 1.27 1.27)
+				)
+				(justify left)
+			)
+		)
+		(pin "Data_B" bidirectional
+			(at 142.24 115.57 180)
+			(effects
+				(font
+					(size 1.27 1.27)
+				)
+				(justify left)
+			)
+		)
 		(instances
 			(project "Buoy PCB"
@@
 			(effects
 				(font
+					(size 1.27 1.27)
+				)
+				(justify right)
+			)
+		)
+		(pin "V_Solar_An" input
+			(at 93.98 105.41 0)
+			(effects
+				(font
+					(size 1.27 1.27)
+				)
+				(justify right)
+			)
+		)
+		(pin "UART0_RX" bidirectional
+			(at 93.98 107.95 0)
+			(effects
+				(font
+					(size 1.27 1.27)
+				)
+				(justify right)
+			)
+		)
+		(pin "UART0_TX" bidirectional
+			(at 93.98 110.49 0)
+			(effects
+				(font
+					(size 1.27 1.27)
+				)
+				(justify right)
+			)
+		)
+		(pin "Data_A" bidirectional
+			(at 93.98 113.03 0)
+			(effects
+				(font
+					(size 1.27 1.27)
+				)
+				(justify right)
+			)
+		)
+		(pin "Data_B" bidirectional
+			(at 93.98 115.57 0)
+			(effects
+				(font
