File: Main PCB KiCAD/Front PCB.kicad_sch (KiCad schematic)
At the start: 0 parts

Commit message: changes adn updates
Parts:
- added D12: RED, LED_SMD:LED_0805_2012Metric_Pad1.15x1.40mm_HandSolder, symbol Device:LED_Small_Filled
- added R8: 1k, Resistor_SMD:R_0805_2012Metric_Pad1.20x1.40mm_HandSolder, symbol Device:R_Small
Connections:
- new net: D12.2 (A), R8.2
- new net GND: D12.1 (K)
- new net Heart Beat: R8.1
Other:
- added sheet RS485 Interface (RS485.kicad_sch)
- added sheet Shrimp (Shrimp.kicad_sch)
- added sheet Solar (solar.kicad_sch)

Commit message: .
Parts:
- added D13: WS2812B, LED_SMD:LED_WS2812B_PLCC4_5.0x5.0mm_P3.2mm, symbol LED:WS2812B
Connections:
- net NeoPixle_Out: now also D13.4 (DIN)
- new net Top PCB +5V: D13.1 (VDD)
- new net Top PCB GND: D13.3 (VSS)
Changed lines of the file:
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@@
+	(wire
+		(pts
+			(xy 245.11 105.41) (xy 252.73 105.41)
+		)
+		(stroke
+			(width 0)
+			(type default)
+		)
+	)
 	(wire
 		(pts
@@
 	(wire
 		(pts
-			(xy 181.61 81.28) (xy 187.96 81.28)
+			(xy 181.61 81.28) (xy 199.39 81.28)
 		)
 		(stroke
@@
 		)
 	)
+	(label "NeoPixle_Out"
+		(at 199.39 81.28 180)
+		(effects
+			(font
+				(size 1.27 1.27)
+			)
+			(justify right bottom)
+		)
+	)
 	(label "Heart Beat"
 		(at 129.54 106.68 180)
@@
 			)
 			(justify left bottom)
+		)
+	)
+	(label "NeoPixle_Out"
+		(at 245.11 105.41 180)
+		(effects
+			(font
+				(size 1.27 1.27)
+			)
+			(justify right bottom)
 		)
 	)
@@
 		)
 	)
-	(hierarchical_label "NeoPixle_Out"
-		(shape output)
-		(at 187.96 81.28 0)
-		(effects
-			(font
-				(size 1.27 1.27)
-			)
-			(justify left)
-		)
-	)
 	(hierarchical_label "Front_PCB_+5V"
 		(shape output)
@@
 			)
 			(justify right)
+		)
+	)
+	(symbol
+		(lib_id "LED:WS2812B")
+		(at 260.35 105.41 0)
+		(unit 1)
+		(exclude_from_sim no)
+		(in_bom yes)
+		(on_board yes)
+		(dnp no)
+		(fields_autoplaced yes)
+		(property "Reference" "D13"
+			(at 271.78 98.9898 0)
+			(effects
+				(font
+					(size 1.27 1.27)
+				)
+			)
+		)
+		(property "Value" "WS2812B"
+			(at 271.78 101.5298 0)
+			(effects
+				(font
+					(size 1.27 1.27)
+				)
+			)
+		)
+		(property "Footprint" "LED_SMD:LED_WS2812B_PLCC4_5.0x5.0mm_P3.2mm"
+			(at 261.62 113.03 0)
+			(effects
+				(font
+					(size 1.27 1.27)
+				)
+				(justify left top)
+				(hide yes)
+			)
+		)
+		(property "Datasheet" "https://cdn-shop.adafruit.com/datasheets/WS2812B.pdf"
+			(at 262.89 114.935 0)
+			(effects
+				(font
+					(size 1.27 1.27)
+				)
+				(justify left top)
+				(hide yes)
+			)
+		)
+		(property "Description" "RGB LED with integrated controller"
+			(at 260.35 105.41 0)
+			(effects
+				(font
+					(size 1.27 1.27)
+				)
+				(hide yes)
+			)
+		)
+		(pin "3"
+		)
+		(pin "1"
+		)
+		(pin "4"
+		)
+		(pin "2"
+		)
+		(instances
+			(project "Buoy PCB"
+				(path "/a041e2a6-7d41-458c-91f3-753821d3dfe9/402c8c5f-ad4a-46d2-a42e-eba9c7fe5855"
+					(reference "D13")
+					(unit 1)
+				)
+			)
 		)
 	)
@@
 					(unit 1)
 				)
+			)
+		)
+	)
+	(symbol
+		(lib_id "power:GND")
+		(at 260.35 113.03 0)
+		(unit 1)
+		(exclude_from_sim no)
+		(in_bom yes)
+		(on_board yes)
+		(dnp no)
+		(fields_autoplaced yes)
+		(property "Reference" "#PWR054"
+			(at 260.35 119.38 0)
+			(effects
+				(font
+					(size 1.27 1.27)
+				)
+				(hide yes)
+			)
+		)
+		(property "Value" "Top PCB GND"
+			(at 260.35 118.11 0)
+			(effects
+				(font
+					(size 1.27 1.27)
+				)
+			)
+		)
+		(property "Footprint" ""
+			(at 260.35 113.03 0)
+			(effects
+				(font
+					(size 1.27 1.27)
+				)
+				(hide yes)
+			)
+		)
+		(property "Datasheet" ""
+			(at 260.35 113.03 0)
+			(effects
+				(font
+					(size 1.27 1.27)
+				)
+				(hide yes)
+			)
+		)
+		(property "Description" ""
+			(at 260.35 113.03 0)
+			(effects
+				(font
+					(size 1.27 1.27)
+				)
+			)
+		)
+		(pin "1"
+		)
+		(instances
+			(project "Buoy PCB"
+				(path "/a041e2a6-7d41-458c-91f3-753821d3dfe9/402c8c5f-ad4a-46d2-a42e-eba9c7fe5855"
+					(reference "#PWR054")
+					(unit 1)
+				)
+			)
+		)
+	)
+	(symbol
+		(lib_id "power:+5V")
+		(at 260.35 97.79 0)
+		(unit 1)
+		(exclude_from_sim no)
+		(in_bom yes)
+		(on_board yes)
+		(dnp no)
+		(fields_autoplaced yes)
+		(property "Reference" "#PWR034"
+			(at 260.35 101.6 0)
+			(effects
+				(font
+					(size 1.27 1.27)
+				)
+				(hide yes)
+			)
+		)
+		(property "Value" "Top PCB +5V"
+			(at 260.35 92.71 0)
+			(effects
+				(font
+					(size 1.27 1.27)
+				)
+			)
+		)
+		(property "Footprint" ""
+			(at 260.35 97.79 0)
+			(effects
+				(font
+					(size 1.27 1.27)
+				)
+				(hide yes)
+			)
+		)
+		(property "Datasheet" ""
+			(at 260.35 97.79 0)
+			(effects
+				(font
+					(size 1.27 1.27)
+				)
+				(hide yes)
+			)
+		)
+		(property "Description" "Power symbol creates a global label with name \"+5V\""
+			(at 260.35 97.79 0)
+			(effects
+				(font
+					(size 1.27 1.27)
+				)
+				(hide yes)
+			)
+		)
+		(pin "1"
+		)
+		(instances
+			(project "Buoy PCB"
+				(path "/a041e2a6-7d41-458c-91f3-753821d3dfe9/402c8c5f-ad4a-46d2-a42e-eba9c7fe5855"
+					(reference "#PWR034")
+					(unit 1)
+				)

Commit message: .
Parts:
- added D14: WS2812B, LED_SMD:LED_WS2812B_PLCC4_5.0x5.0mm_P3.2mm, symbol LED:WS2812B
Connections:
- net Top PCB +5V: now also D14.1 (VDD)
- net Top PCB GND: now also D14.3 (VSS)
- net at D13.2 (DOUT): now also D14.4 (DIN)
- new net NeoPixle_Connect_out: D14.2 (DOUT)
Other:
- moved on the sheet: D13

Commit message: .
Parts:
- added U3: Pimoroni PGA2350, KiCad Footprints:PGA2350, symbol KiCad Symbols:Pimoroni PGA2350
Connections:
- net Heart Beat: now also U3.13 (GP0)
- net NeoPixle_Out: now also U3.31 (GP39)
- net V_Solar_An: now also U3.32 (GP40/ADC0)
- new net: U3.1 (GND), U3.10 (GND), U3.12 (GND), U3.19 (GND), U3.55 (GND), U3.64 (GND)
Other:
- removed sheet Shrimp

Commit message: .
Parts:
- added D17: 20V 1A, Diode_SMD:D_0805_2012Metric_Pad1.15x1.40mm_HandSolder, symbol Device:D_Schottky_Filled
- added J5: USB_B, symbol Connector:USB_B
- added SW2: Reset, Button_Switch_THT:SW_PUSH-12mm, symbol Switch:SW_Push
- added SW3: Boot, Button_Switch_THT:SW_PUSH-12mm, symbol Switch:SW_Push
Connections:
- net Top PCB GND is gone; now on net Front PCB GND: D13.3 (VSS), D14.3 (VSS)
- net Front PCB GND: now also D12.1 (K), U3.1 (GND), U3.10 (GND), U3.12 (GND), U3.19 (GND), U3.55 (GND), U3.64 (GND)
- net GND: now also J5.4 (GND), SW2.2, SW3.2; no longer D12.1 (K)
- net Heart Beat: no longer U3.13 (GP0)
- net NeoPixle_Out: now also U3.41 (GP14); no longer U3.31 (GP39)
- net UART1_TX: now reaches U3.11 (GP2)
- net UART0_RX: now reaches U3.2 (GP1)
- net UART1_RX: now reaches U3.21 (GP4)
- net UART1_TX_EN: now reaches U3.22 (GP3)
- net +5V: now reaches U3.3 (VBUS)
- net +5V: now also D17.1 (K)
- net at U3.5 (RUN): now also SW2.1
- net at U3.6 (USB_D+): now also J5.3 (D+)
- net at U3.7 (USB_D-): now also J5.2 (D-)
- net at U3.8 (BOOTSEL): now also SW3.1
- new net: D17.2 (A), J5.1 (VBUS)
- new net UART0_TX: U3.13 (GP0)

Commit message: .
Parts:
- removed J5: USB_B, symbol Connector:USB_B
- removed SW2: Reset, Button_Switch_THT:SW_PUSH-12mm, symbol Switch:SW_Push
- removed SW3: Boot, Button_Switch_THT:SW_PUSH-12mm, symbol Switch:SW_Push
- removed U3: Pimoroni PGA2350, KiCad Footprints:PGA2350, symbol KiCad Symbols:Pimoroni PGA2350
- added A1: Adafruit_Feather_M0_RFM9x_LoRa_Radio, Module:Adafruit_Feather_M0_RFM, symbol MCU_Module:Adafruit_Feather_M0_RFM9x_LoRa_Radio
- added J9: Conn_01x02, Connector_JST:JST_EH_S2B-EH_1x02_P2.50mm_Horizontal, symbol Connector_Generic:Conn_01x02
Connections:
- net Front PCB GND is gone; now on net GND: D12.1 (K), D13.3 (VSS), D14.3 (VSS)
- net Top PCB +5V is gone; now on net +5V: D13.1 (VDD), D14.1 (VDD)
- net +5V: now also A1.26 (USB)
- net GND: now also A1.4 (GND), J9.2 (Pin_2)
- net Heart Beat: now also A1.20 (D6)
- net NeoPixle_Out: now also A1.19 (D5)
- net V_Solar_An: now also A1.5 (DAC0/A0)
- net at D17.2 (A): now also J9.1 (Pin_1)
Other:
- removed sheet Solar
- moved on the sheet: D17

Commit message: .
Parts:
- added BT1, BT2: Battery_Cell, Battery:BatteryHolder_Keystone_1042_1x18650, symbol Device:Battery_Cell
- J9: value Conn_01x02 -> BenchTop Power
Connections:
- net GND: now also BT1.2 (-), BT2.2 (-)
- net UART0_RX: now also A1.14 (RX/D0)
- net UART0_TX: now also A1.15 (TX/D1)
- net UART1_RX: now also A1.23 (D11)
- net UART1_TX: now also A1.24 (D12)
- net UART1_TX_EN: now also A1.22 (D10)
- net +Bat: now reaches A1.28 (VBAT)
- net +Bat: now also BT1.1 (+), BT2.1 (+)
- no-connect marks 0 -> 1
Other:
- note added: "(Ain Battery)"
- note added: "https://learn.adafruit.com/assets/113562"
- moved on the sheet: D12, R8

Commit message: .
Parts:
- removed A1: Adafruit_Feather_M0_RFM9x_LoRa_Radio, Module:Adafruit_Feather_M0_RFM, symbol MCU_Module:Adafruit_Feather_M0_RFM9x_LoRa_Radio
Changed lines of the file:
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@@
-	)
-	(symbol
-		(lib_id "MCU_Module:Adafruit_Feather_M0_RFM9x_LoRa_Radio")
-		(at 92.71 91.44 0)
-		(unit 1)
-		(body_style 1)
-		(exclude_from_sim no)
-		(in_bom yes)
-		(on_board yes)
-		(in_pos_files yes)
-		(dnp no)
-		(fields_autoplaced yes)
-		(property "Reference" "A1"
-			(at 94.8533 124.46 0)
-			(show_name no)
-			(do_not_autoplace no)
-			(effects
-				(font
-					(size 1.27 1.27)
-				)
-				(justify left)
-			)
-		)
-		(property "Value" "Adafruit_Feather_M0_RFM9x_LoRa_Radio"
-			(at 94.8533 127 0)
-			(show_name no)
-			(do_not_autoplace no)
-			(effects
-				(font
-					(size 1.27 1.27)
-				)
-				(justify left)
-			)
-		)
-		(property "Footprint" "Module:Adafruit_Feather_M0_RFM"
-			(at 95.25 125.73 0)
-			(hide yes)
-			(show_name no)
-			(do_not_autoplace no)
-			(effects
-				(font
-					(size 1.27 1.27)
-				)
-				(justify left)
-			)
-		)
-		(property "Datasheet" "https://cdn-learn.adafruit.com/downloads/pdf/adafruit-feather-m0-radio-with-lora-radio-module.pdf"
-			(at 92.71 111.76 0)
-			(hide yes)
-			(show_name no)
-			(do_not_autoplace no)
-			(effects
-				(font
-					(size 1.27 1.27)
-				)
-			)
-		)
-		(property "Description" "Microcontroller module with SAMD21 Cortex-M0 MCU and RFM9x Radio"
-			(at 92.71 91.44 0)
-			(hide yes)
-			(show_name no)
-			(do_not_autoplace no)
-			(effects
-				(font
-					(size 1.27 1.27)
-				)
-			)
-		)
-		(pin "4"
-		)
-		(pin "13"
-		)
-		(pin "6"
-		)
-		(pin "1"
-		)
-		(pin "7"
-		)
-		(pin "8"
-		)
-		(pin "10"
-		)
-		(pin "19"
-		)
-		(pin "25"
-		)
-		(pin "15"
-		)
-		(pin "2"
-		)
-		(pin "3"
-		)
-		(pin "5"
-		)
-		(pin "9"
-		)
-		(pin "11"
-		)
-		(pin "12"
-		)
-		(pin "16"
-		)
-		(pin "17"
-		)
-		(pin "18"
-		)
-		(pin "20"
-		)
-		(pin "21"
-		)
-		(pin "22"
-		)
-		(pin "23"
-		)
-		(pin "14"
-		)
-		(pin "24"
-		)
-		(pin "29"
-		)
-		(pin "27"
-		)
-		(pin "31"
-		)
-		(pin "26"
-		)
-		(pin "30"
-		)
-		(pin "32"
-		)
-		(pin "28"
-		)
-		(instances
-			(project "Buoy PCB"
-				(path "/a041e2a6-7d41-458c-91f3-753821d3dfe9/402c8c5f-ad4a-46d2-a42e-eba9c7fe5855"
-					(reference "A1")
-					(unit 1)
-				)
-			)
-		)
 	)
 	(symbol
