File: Main PCB KiCAD/Front PCB.kicad_sch (KiCad schematic)
At the start: 8 parts, among them J9 BenchTop Power

Commit message: .
Parts:
- added U1: (no value), symbol KiCad Symbols:Heltec WiFi LoRa 32
Connections:
- net +5V: now also U1.35 (5V)
- net GND: now also U1.1 (GND), U1.36 (GND)
- net Heart Beat: now also U1.7 (GPIO42)
- net NeoPixle_Out: now also U1.6 (GPIO46)
- net UART0_RX: now also U1.32 (GPIO44/U0_RXD)
- net UART0_TX: now also U1.31 (GPIO43/U0_TXD)
- net UART1_RX: now also U1.10 (GPIO39)
- net UART1_TX: now also U1.11 (GPIO38)
- net UART1_TX_EN: now also U1.9 (GPIO40)
- net V_Solar_An: now also U1.13 (GPIO2/ADC1_CH1)
- new net: U1.2 (3V3), U1.3 (3V3)
- new net: U1.33 (Ve), U1.34 (Ve)
Other:
- note removed: "https://learn.adafruit.com/assets/113562"
