File: Main PCB KiCAD/Back PCB.kicad_sch (KiCad schematic)
At the start: 0 parts

Commit message: .
Parts:
- added D15, D16: WS2812B, LED_SMD:LED_WS2812B_PLCC4_5.0x5.0mm_P3.2mm, symbol LED:WS2812B
Connections:
- net Back PCB +5V: now also D15.1 (VDD), D16.1 (VDD)
- net Back PCB GND: now also D15.3 (VSS), D16.3 (VSS)
- new net: D15.2 (DOUT), D16.4 (DIN)
- new net NeoPixle_Connect_in: D15.4 (DIN)

Commit message: .
Connections:
- net Back PCB +5V renamed +5V
- net Back PCB GND renamed GND
Other:
- added sheet Solar (solar.kicad_sch)
Changed lines of the file:
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@@
 	(wire
 		(pts
-			(xy 35.56 25.4) (xy 34.29 25.4)
+			(xy 248.92 36.83) (xy 251.46 36.83)
 		)
 		(stroke
@@
 	(wire
 		(pts
-			(xy 35.56 24.13) (xy 35.56 25.4)
-		)
-		(stroke
-			(width 0)
-			(type default)
-		)
-	)
-	(wire
-		(pts
-			(xy 35.56 38.1) (xy 35.56 39.37)
-		)
-		(stroke
-			(width 0)
-			(type default)
-		)
-	)
-	(wire
-		(pts
 			(xy 102.87 20.32) (xy 102.87 22.86)
-		)
-		(stroke
-			(width 0)
-			(type default)
-		)
-	)
-	(wire
-		(pts
-			(xy 34.29 38.1) (xy 35.56 38.1)
 		)
 		(stroke
@@
 		)
 	)
-	(hierarchical_label "Back_PCB_GND"
-		(shape input)
-		(at 34.29 38.1 180)
+	(hierarchical_label "V_Solar_An"
+		(shape output)
+		(at 251.46 36.83 0)
 		(effects
 			(font
 				(size 1.27 1.27)
 			)
-			(justify right)
-		)
-	)
-	(hierarchical_label "Back_PCB_+5V"
-		(shape input)
-		(at 34.29 25.4 180)
-		(effects
-			(font
-				(size 1.27 1.27)
-			)
-			(justify right)
+			(justify left)
 		)
 	)
@@
 		(lib_id "power:GND")
 		(at 80.01 40.64 0)
+		(mirror y)
 		(unit 1)
 		(body_style 1)
@@
 			)
 		)
-		(property "Value" "Back PCB GND"
+		(property "Value" "GND"
 			(at 80.01 45.72 0)
 			(show_name no)
@@
 			)
 		)
-		(property "Description" ""
+		(property "Description" "Power symbol creates a global label with name \"GND\" , ground"
 			(at 80.01 40.64 0)
+			(hide yes)
 			(show_name no)
 			(do_not_autoplace no)
@@
 	(symbol
 		(lib_id "power:GND")
-		(at 35.56 39.37 0)
+		(at 102.87 40.64 0)
+		(mirror y)
 		(unit 1)
 		(body_style 1)
@@
 		(dnp no)
 		(fields_autoplaced yes)
-		(property "Reference" "#PWR051"
-			(at 35.56 45.72 0)
-			(hide yes)
-			(show_name no)
-			(do_not_autoplace no)
-			(effects
-				(font
-					(size 1.27 1.27)
-				)
-			)
-		)
-		(property "Value" "Back PCB GND"
-			(at 35.56 44.45 0)
+		(property "Reference" "#PWR058"
+			(at 102.87 46.99 0)
+			(hide yes)
+			(show_name no)
+			(do_not_autoplace no)
+			(effects
+				(font
+					(size 1.27 1.27)
+				)
+			)
+		)
+		(property "Value" "GND"
+			(at 102.87 45.72 0)
 			(show_name no)
 			(do_not_autoplace no)
@@
 		)
 		(property "Footprint" ""
-			(at 35.56 39.37 0)
+			(at 102.87 40.64 0)
 			(hide yes)
 			(show_name no)
@@
 		)
 		(property "Datasheet" ""
-			(at 35.56 39.37 0)
-			(hide yes)
-			(show_name no)
-			(do_not_autoplace no)
-			(effects
-				(font
-					(size 1.27 1.27)
-				)
-			)
-		)
-		(property "Description" ""
-			(at 35.56 39.37 0)
+			(at 102.87 40.64 0)
+			(hide yes)
+			(show_name no)
+			(do_not_autoplace no)
+			(effects
+				(font
+					(size 1.27 1.27)
+				)
+			)
+		)
+		(property "Description" "Power symbol creates a global label with name \"GND\" , ground"
+			(at 102.87 40.64 0)
+			(hide yes)
 			(show_name no)
 			(do_not_autoplace no)
@@
 			(project "Buoy PCB"
 				(path "/a041e2a6-7d41-458c-91f3-753821d3dfe9/2b71a53e-4a43-4bc8-a314-937e96c041a6"
-					(reference "#PWR051")
-					(unit 1)
-				)
-			)
-		)
-	)
-	(symbol
-		(lib_id "power:GND")
-		(at 102.87 40.64 0)
-		(unit 1)
-		(body_style 1)
-		(exclude_from_sim no)
-		(in_bom yes)
-		(on_board yes)
-		(in_pos_files yes)
-		(dnp no)
-		(fields_autoplaced yes)
-		(property "Reference" "#PWR057"
-			(at 102.87 46.99 0)
-			(hide yes)
-			(show_name no)
-			(do_not_autoplace no)
-			(effects
-				(font
-					(size 1.27 1.27)
-				)
-			)
-		)
-		(property "Value" "Back PCB GND"
-			(at 102.87 45.72 0)
-			(show_name no)
-			(do_not_autoplace no)
-			(effects
-				(font
-					(size 1.27 1.27)
-				)
-			)
-		)
-		(property "Footprint" ""
-			(at 102.87 40.64 0)
-			(hide yes)
-			(show_name no)
-			(do_not_autoplace no)
-			(effects
-				(font
-					(size 1.27 1.27)
-				)
-			)
-		)
-		(property "Datasheet" ""
-			(at 102.87 40.64 0)
-			(hide yes)
-			(show_name no)
-			(do_not_autoplace no)
-			(effects
-				(font
-					(size 1.27 1.27)
-				)
-			)
-		)
-		(property "Description" ""
-			(at 102.87 40.64 0)
-			(show_name no)
-			(do_not_autoplace no)
-			(effects
-				(font
-					(size 1.27 1.27)
-				)
-			)
-		)
-		(pin "1"
-		)
-		(instances
-			(project "Buoy PCB"
-				(path "/a041e2a6-7d41-458c-91f3-753821d3dfe9/2b71a53e-4a43-4bc8-a314-937e96c041a6"
-					(reference "#PWR057")
-					(unit 1)
-				)
-			)
-		)
-	)
-	(symbol
-		(lib_id "power:+5V")
-		(at 35.56 24.13 0)
-		(unit 1)
-		(body_style 1)
-		(exclude_from_sim no)
-		(in_bom yes)
-		(on_board yes)
-		(in_pos_files yes)
-		(dnp no)
-		(fields_autoplaced yes)
-		(property "Reference" "#PWR050"
-			(at 35.56 27.94 0)
-			(hide yes)
-			(show_name no)
-			(do_not_autoplace no)
-			(effects
-				(font
-					(size 1.27 1.27)
-				)
-			)
-		)
-		(property "Value" "Back PCB +5V"
-			(at 35.56 19.05 0)
-			(show_name no)
-			(do_not_autoplace no)
-			(effects
-				(font
-					(size 1.27 1.27)
-				)
-			)
-		)
-		(property "Footprint" ""
-			(at 35.56 24.13 0)
-			(hide yes)
-			(show_name no)
-			(do_not_autoplace no)
-			(effects
-				(font
-					(size 1.27 1.27)
-				)
-			)
-		)
-		(property "Datasheet" ""
-			(at 35.56 24.13 0)
-			(hide yes)
-			(show_name no)
-			(do_not_autoplace no)
-			(effects
-				(font
-					(size 1.27 1.27)
-				)
-			)
-		)
-		(property "Description" "Power symbol creates a global label with name \"+5V\""
-			(at 35.56 24.13 0)
-			(hide yes)
-			(show_name no)
-			(do_not_autoplace no)
-			(effects
-				(font
-					(size 1.27 1.27)
-				)
-			)
-		)
-		(pin "1"
-		)
-		(instances
-			(project "Buoy PCB"
-				(path "/a041e2a6-7d41-458c-91f3-753821d3dfe9/2b71a53e-4a43-4bc8-a314-937e96c041a6"
-					(reference "#PWR050")
+					(reference "#PWR058")
 					(unit 1)
 				)
@@
 		(dnp no)
 		(fields_autoplaced yes)
-		(property "Reference" "#PWR059"
+		(property "Reference" "#PWR055"
 			(at 80.01 24.13 0)
 			(hide yes)
@@
 			)
 		)
-		(property "Value" "Back PCB +5V"
-			(at 80.01 15.24 0)
-			(show_name no)
-			(do_not_autoplace no)
-			(effects
-				(font
-					(size 1.27 1.27)
-				)
+		(property "Value" "+5V"
+			(at 82.55 19.0499 0)
+			(show_name no)
+			(do_not_autoplace no)
+			(effects
+				(font
+					(size 1.27 1.27)
+				)
+				(justify left)
 			)
 		)
@@
 			(project "Buoy PCB"
 				(path "/a041e2a6-7d41-458c-91f3-753821d3dfe9/2b71a53e-4a43-4bc8-a314-937e96c041a6"
-					(reference "#PWR059")
+					(reference "#PWR055")
 					(unit 1)
 				)
@@
 		(dnp no)
 		(fields_autoplaced yes)
-		(property "Reference" "#PWR060"
+		(property "Reference" "#PWR057"
 			(at 102.87 24.13 0)
 			(hide yes)
@@
 			)
 		)
-		(property "Value" "Back PCB +5V"
-			(at 102.87 15.24 0)
-			(show_name no)
-			(do_not_autoplace no)
-			(effects
-				(font
-					(size 1.27 1.27)
-				)
+		(property "Value" "+5V"
+			(at 105.41 19.0499 0)
+			(show_name no)
+			(do_not_autoplace no)
+			(effects
+				(font
+					(size 1.27 1.27)
+				)
+				(justify left)
 			)
 		)
@@
 			(project "Buoy PCB"
 				(path "/a041e2a6-7d41-458c-91f3-753821d3dfe9/2b71a53e-4a43-4bc8-a314-937e96c041a6"
-					(reference "#PWR060")
+					(reference "#PWR057")
 					(unit 1)
 				)
 			)
+		)
+	)
+	(sheet
+		(at 215.9 35.56)
+		(size 33.02 15.24)
+		(exclude_from_sim no)
+		(in_bom yes)
+		(on_board yes)
+		(dnp no)
+		(fields_autoplaced yes)
+		(stroke
+			(width 0.1524)
+			(type solid)
+		)
+		(fill
+			(color 0 0 0 0)
+		)
+		(property "Sheetname" "Solar"
+			(at 215.9 34.8484 0)
+			(show_name no)
+			(do_not_autoplace no)
+			(effects
+				(font
+					(size 1.27 1.27)
+				)
+				(justify left bottom)
+			)
+		)
+		(property "Sheetfile" "solar.kicad_sch"
+			(at 215.9 51.3846 0)
+			(hide yes)
+			(show_name no)
+			(do_not_autoplace no)
+			(effects
+				(font
+					(size 1.27 1.27)
+				)
+				(justify left top)
+			)
+		)
+		(pin "V_Solar_An" output
+			(at 248.92 36.83 0)
+			(effects
+				(font
+					(size 1.27 1.27)
+				)
+				(justify right)
+			)
+		)
+		(instances
+			(project "Buoy PCB"
+				(path "/a041e2a6-7d41-458c-91f3-753821d3dfe9/2b71a53e-4a43-4bc8-a314-937e96c041a6"
+					(page "2")
+				)
+			)

Commit message: .
Parts:
- added C8: 0.1uF, Capacitor_SMD:C_0805_2012Metric_Pad1.18x1.45mm_HandSolder, symbol Device:C_Small
- added C9: 47μF, Capacitor_SMD:CP_Elec_5x5.9, symbol Device:C_Polarized_Small
Connections:
- net +5V: now also C8.2, C9.1
- net GND: now also C8.1, C9.2

Commit message: .
Parts:
- added J10: RS485 Addr 0, Connector_JST:JST_EH_S7B-EH_1x07_P2.50mm_Horizontal, symbol Connector_Generic:Conn_01x07
- added J11: RS485 Addr 1, Connector_JST:JST_EH_S7B-EH_1x07_P2.50mm_Horizontal, symbol Connector_Generic:Conn_01x07
- added J12: RS485 Addr 2, Connector_JST:JST_EH_S7B-EH_1x07_P2.50mm_Horizontal, symbol Connector_Generic:Conn_01x07
Connections:
- net +5V: now also J10.1 (Pin_1), J11.1 (Pin_1), J12.1 (Pin_1)
- net Data_A: now also J10.6 (Pin_6), J11.6 (Pin_6), J12.6 (Pin_6)
- net Data_B: now also J10.7 (Pin_7), J11.7 (Pin_7), J12.7 (Pin_7)
- net GND: now also J10.2 (Pin_2), J10.3 (Pin_3), J10.4 (Pin_4), J10.5 (Pin_5), J11.2 (Pin_2), J11.4 (Pin_4), J11.5 (Pin_5), J12.2 (Pin_2), J12.3 (Pin_3), J12.5 (Pin_5)
- no-connect marks 0 -> 2
