File: Main PCB KiCAD/Assets/SubPCBs/Shrimps/Shrimp ATmega328P-P.kicad_sch (KiCad schematic)
At the start: 22 parts, among them J1 UART, J2 ICSP, J3 I2C, U1 ATmega328P-P, Y1 16 MHz

Commit message: update
Parts:
- renumbered C3 to C1, C4 to C2, C6 to C3, C5 to C4, C1 to C5, C2 to C6, J1 to J5, J2 to J6, J3 to J7, R5 to R1, R4 to R2, R2 to R3, R3 to R4, R6 to R5, R1 to R6, TP3 to TP1, TP1 to TP2, TP2 to TP3
