File: Sub PCB KiCAD/Sub PCB.kicad_sch (KiCad schematic)
At the start: 10 parts

Commit message: .
Parts:
- added A1: RaspberryPi_Pico, Module:RaspberryPi_Pico_Common_Unspecified, symbol MCU_Module:RaspberryPi_Pico
- added R8: 10k, Resistor_SMD:R_0805_2012Metric_Pad1.20x1.40mm_HandSolder, symbol Device:R_Small
- added R9: 2.2k, Resistor_SMD:R_0805_2012Metric_Pad1.20x1.40mm_HandSolder, symbol Device:R_Small
Connections:
- net +12V: now also R8.2
- net +5V: now also A1.40 (VBUS); no longer D1.2 (K), D2.2 (K), R4.2, R6.2
- net ADDR_1: now also A1.31 (GPIO26_ADC0)
- net ADDR_2: now also A1.32 (GPIO27_ADC1)
- net GND: now also A1.13 (GND), A1.18 (GND), A1.23 (GND), A1.28 (GND), A1.3 (GND), A1.38 (GND), A1.8 (GND), R9.1
- new net +3V3: D1.2 (K), D2.2 (K), R4.2, R6.2
- new net UART0_RX: A1.2 (GPIO1)
- new net UART0_TX: A1.1 (GPIO0)
- new net UART1_RX: A1.7 (GPIO5)
- new net UART1_TX: A1.6 (GPIO4)
- new net V_Supply: A1.34 (GPIO28_ADC2), R8.1, R9.2
- no-connect marks 0 -> 2
Other:
- note added: "https://datacapturecontrol.com/articles/io-devices/microcontrollers/rpi-pico"

Commit message: .
Parts:
- removed A1: RaspberryPi_Pico, Module:RaspberryPi_Pico_Common_Unspecified, symbol MCU_Module:RaspberryPi_Pico
- added A1: Arduino_UNO_R3, Module:Arduino_UNO_R3, symbol MCU_Module:Arduino_UNO_R3
- added J2: ~, Connector_PinHeader_2.54mm:PinHeader_1x04_P2.54mm_Vertical, symbol Connector:Conn_01x04_Pin
- added R10: 10k, Resistor_SMD:R_0805_2012Metric_Pad1.20x1.40mm_HandSolder, symbol Device:R_Small
- J1: footprint (none) -> Connector_PinHeader_2.54mm:PinHeader_1x07_P2.54mm_Vertical
Connections:
- net +3V3 is gone; now on net +5V: D1.2 (K), D2.2 (K), R4.2, R6.2
- net +12V: now also A1.8 (VIN)
- net +5V: now also A1.5 (+5V), J2.2 (Pin_2)
- net ADDR_1: now also A1.10 (A1)
- net ADDR_2: now also A1.11 (A2)
- net GND: now also A1.29 (GND), A1.6 (GND), A1.7 (GND), J2.1 (Pin_1)
- net RS485_A: now also J1.6 (Pin_6); no longer J1.5 (Pin_5)
- net RS485_B: now also J1.5 (Pin_5); no longer J1.6 (Pin_6)
- net UART0_RX: now also A1.16 (D1/TX)
- net UART0_TX: now also A1.15 (D0/RX)
- net UART1_RX: now also A1.19 (D4)
- net UART1_TX: now also A1.17 (D2)
- net V_Supply: now also A1.9 (A0), R10.1; no longer R8.1, R9.2
- new net: R10.2, R8.1, R9.2
- new net I2C_SCL: A1.14 (SCL/A5), J2.4 (Pin_4)
- new net I2C_SDA: A1.13 (SDA/A4), J2.3 (Pin_3)
- new net UART1_TX_EN: A1.18 (D3)
- no-connect marks 2 -> 1
Other:
- added sheet RS485_UART (RS485_UART.kicad_sch)
- note removed: "https://datacapturecontrol.com/articles/io-devices/microcontrollers/rpi-pico"

Commit message: .
Parts:
- removed A1: Arduino_UNO_R3, Module:Arduino_UNO_R3, symbol MCU_Module:Arduino_UNO_R3
- added U2: Pimoroni PGA2350, Skippy's:PGA2350, symbol Skippy's:Pimoroni PGA2350
Connections:
- net +5V: now also U2.3 (VBUS); no longer D1.2 (K), D2.2 (K), J2.2 (Pin_2), R4.2, R6.2
- net ADDR_1: now also U2.28 (GP42/ADC2)
- net ADDR_2: now also U2.27 (GP41/ADC1)
- net GND: now also U2.1 (GND), U2.10 (GND), U2.12 (GND), U2.19 (GND), U2.55 (GND), U2.64 (GND)
- net I2C_SCL: now also U2.20 (GP45/ADC5)
- net I2C_SDA: now also U2.24 (GP44/ADC4)
- net UART0_RX: now also U2.2 (GP1)
- net UART0_TX: now also U2.13 (GP0)
- net UART1_RX: now also U2.21 (GP4)
- net UART1_TX: now also U2.11 (GP2)
- net UART1_TX_EN: now also U2.22 (GP3)
- net V_Supply: now also U2.32 (GP40/ADC0)
- new net +3V3: D1.2 (K), D2.2 (K), J2.2 (Pin_2), R4.2, R6.2
- no-connect marks 1 -> 0

Commit message: .
Parts:
- D1, D2: footprint Package_TO_SOT_SMD:SOT-23_Handsoldering -> Package_TO_SOT_SMD:SOT-23; symbol Diode:BAT54S -> KiCad Symbols:BAT54S
- J1, J2: value ~ -> (none)
- U1: renamed from U2; footprint Skippy's:PGA2350 -> LED Cube:PGA2350; symbol Skippy's:Pimoroni PGA2350 -> KiCad Symbols:Pimoroni PGA2350
- renumbered R8 to R1, R7 to R10, R9 to R2, R1 to R3, R2 to R4, R3 to R5, R10 to R6, R4 to R7, R5 to R8, R6 to R9
