File: Sub PCB KiCAD/Sub PCB.kicad_sch (KiCad schematic)
At the start: 15 parts, among them U1 Pimoroni PGA2350

Commit message: .
Parts:
- added D3, D4: 20V 1A, Diode_SMD:D_0805_2012Metric_Pad1.15x1.40mm_HandSolder, symbol Device:D_Schottky_Filled
- added D5: Power, LED_SMD:LED_0805_2012Metric_Pad1.15x1.40mm_HandSolder, symbol Device:LED_Small_Filled
- added J3: USB_B, symbol Connector:USB_B
- added R17: 520, Resistor_SMD:R_0805_2012Metric_Pad1.20x1.40mm_HandSolder, symbol Device:R_Small
- added SW1: Reset, Button_Switch_THT:SW_PUSH-12mm, symbol Switch:SW_Push
- added SW2: Boot, Button_Switch_THT:SW_PUSH-12mm, symbol Switch:SW_Push
Connections:
- net +12V: now also D4.1 (K), D5.2 (A); no longer J1.1 (Pin_1)
- net +5V: now also D3.1 (K)
- net GND: now also J3.4 (GND), R17.1, SW1.2, SW2.2
- net at U1.5 (RUN): now also SW1.1
- net at U1.6 (USB_D+): now also J3.3 (D+)
- net at U1.7 (USB_D-): now also J3.2 (D-)
- net at U1.8 (BOOTSEL): now also SW2.1
- new net: D3.2 (A), J3.1 (VBUS)
- new net: D5.1 (K), R17.2
- new net: D4.2 (A), J1.1 (Pin_1)
Other:
- moved on the sheet: R1, R2, R6

Commit message: .
Parts:
- U1: footprint LED Cube:PGA2350 -> KiCad Footprints:PGA2350
Changed lines of the file:
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@@
 			)
 		)
-		(property "Footprint" "LED Cube:PGA2350"
+		(property "Footprint" "KiCad Footprints:PGA2350"
 			(at 179.07 162.052 0)
 			(hide yes)
@@
 			)
 		)
-		(property "Datasheet" "https://docs.arduino.cc/resources/datasheets/ABX00053-datasheet.pdf"
+		(property "Datasheet" "https://shop.pimoroni.com/products/pga2350"
 			(at 204.47 159.512 0)
 			(hide yes)
@@
 			)
 		)
-		(property "Description" "Arduino Nano board based on the RP2040 microcontroller with a dual-core 133 MHz ARM Cortex-M0+ processor, 264 kB SRAM, and up to 16 MB flash memory. Operates at 3.3V, with 5V Micro USB input and 4-20V VIN. Features Wi-Fi®, Bluetooth® LE, digital and analog pins, and supports SPI, I2C, UART, and PIO. Includes a 6-axis IMU, RGB LED, microphone, and cryptographic chip for secure communication."
+		(property "Description" "A minimal but powerful RP2350 breakout board modelled on a Pin Grid Array, with the maximum exposed pins crammed into the smallest possible space."
 			(at 374.396 156.972 0)
 			(hide yes)
