File: Sub PCB KiCAD/RS485_UART.kicad_sch (KiCad schematic)
At the start: 7 parts, among them U1 MAX485E

Commit message: .
Connections:
- net +5V renamed +3V3

Commit message: .
Parts:
- renumbered R15 to R11, R16 to R12, R11 to R13, R12 to R14, R13 to R15, R14 to R16, U1 to U2

Commit message: .
Changed lines of the file:
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@@
 			(effects
 				(font
-					(size 1.27 1.27)
+					(size 1.016 1.016)
 				)
 				(justify right)
@@
 			(effects
 				(font
-					(size 1.27 1.27)
+					(size 1.016 1.016)
 				)
 				(justify right)
